Commit message: doc:升级ROS21.6.0版本，主要修改项：1添加RML63III型标识，2添加三代modbus接口，3rm_driver doc中添加相关说明，4rm_driver config添加udp相关配置，5部分其他接口。

File: rm_description/urdf/rml_63.urdf (robot description, URDF)
Before this commit: robot rml_63_description, 7 links, 6 joints
Links:
- link base_link: mass 1.6314 -> 0.66248
Joints:
- joint joint1: origin xyz=0 0 0.1625 rpy=0 0 0 -> xyz=0 0 0.172 rpy=0 0 0

File: rm_description/urdf/rml_63.urdf.xacro (robot description, xacro)
@@ -3,6 +3,9 @@
     <!-- link6_type -->
     <xacro:arg name="link6_type" default="Link6" />
+    <xacro:arg name="base_type" default="base_link" />
     <!-- arg->property -->
     <xacro:property name="link6_type" value="$(arg link6_type)" />
+    <xacro:property name="base_type" value="$(arg base_type)" />
+    <xacro:if value="${ base_type =='base_link' }">
     <link
     name="base_link">
@@ -89,4 +92,104 @@
     type="revolute">
     <origin
+      xyz="0 0 0.172"
+      rpy="0 0 0" />
+    <parent
+      link="base_link" />
+    <child
+      link="link1" />
+    <axis
+      xyz="0 0 1" />
+    <limit
+      lower="-3.107"
+      upper="3.107"
+      effort="100"
+      velocity="1" />
+  </joint>
+  </xacro:if>
+<xacro:if value="${ base_type =='base_link_III' }">
+    <link
+    name="base_link">
+    <inertial>
+      <origin
+        xyz="0.000204933302096124 -8.24661684233942E-05 0.0435919339026087"
+        rpy="0 0 0" />
+      <mass
+        value="0.604237569846431" />
+      <inertia
+        ixx="0.00082415777403083"
+        ixy="2.9270718368632E-06"
+        ixz="-2.8722520476522E-05"
+        iyy="0.000820579526371655"
+        iyz="2.21535061552891E-06"
+        izz="0.000685679517381249" />
+    </inertial>
+    <visual>
+      <origin
+        xyz="0 0 0"
+        rpy="0 0 0" />
+      <geometry>
+        <mesh
+          filename="package://rm_description/meshes/rm_63_arm/base_link_III.STL" />
+      </geometry>
+      <material
+        name="">
+        <color
+          rgba="0.792156862745098 0.819607843137255 0.933333333333333 1" />
+      </material>
+    </visual>
+    <collision>
+      <origin
+        xyz="0 0 0"
+        rpy="0 0 0" />
+      <geometry>
+        <mesh
+          filename="package://rm_description/meshes/rm_63_arm/base_link_III.STL" />
+      </geometry>
+    </collision>
+  </link>
+  <link
+    name="link1">
+    <inertial>
+      <origin
+        xyz="-0.030909 -0.0013023 -0.0053121"
+        rpy="0 0 0" />
+      <mass
+        value="1.7668" />
+      <inertia
+        ixx="0.0014534"
+        ixy="-0.00017578"
+        ixz="0.0002802"
+        iyy="0.0043772"
+        iyz="1.7209E-05"
+        izz="0.0040911" />
+    </inertial>
+    <visual>
+      <origin
+        xyz="0 0 0"
+        rpy="0 0 0" />
+      <geometry>
+        <mesh
+          filename="package://rm_description/meshes/rm_63_arm/link1_III.STL" />
+      </geometry>
+      <material
+        name="">
+        <color
+          rgba="1 1 1 1" />
+      </material>
+    </visual>
+    <collision>
+      <origin
+        xyz="0 0 0"
+        rpy="0 0 0" />
+      <geometry>
+        <mesh
+          filename="package://rm_description/meshes/rm_63_arm/link1_III.STL" />
+      </geometry>
+    </collision>
+  </link>
+  <joint
+    name="joint1"
+    type="revolute">
+    <origin
       xyz="0 0 0.1625"
       rpy="0 0 0" />
@@ -103,4 +206,5 @@
       velocity="1" />
   </joint>
+  </xacro:if>
   <link
     name="link2">

File: rm_description/urdf/rml_63_gazebo.urdf.xacro (robot description, xacro)
@@ -3,6 +3,9 @@
     <!-- link6_type -->
     <xacro:arg name="link6_type" default="Link6" />
+    <xacro:arg name="base_type" default="base_link" />
     <!-- arg->property -->
     <xacro:property name="link6_type" value="$(arg link6_type)" />
+    <xacro:property name="base_type" value="$(arg base_type)" />
+    <xacro:if value="${ base_type =='base_link' }">
     <link
     name="base_link">
@@ -13,4 +16,203 @@
       <mass
         value="1.6314" />
+      <inertia
+        ixx="0.0022252"
+        ixy="7.9005E-06"
+        ixz="-7.7558E-05"
+        iyy="0.0022156"
+        iyz="5.9846E-06"
+        izz="0.0018513" />
+    </inertial>
+    <visual>
+      <origin
+        xyz="0 0 0"
+        rpy="0 0 0" />
+      <geometry>
+        <mesh
+          filename="file://$(find rm_description)/meshes/rm_63_arm/base_link.STL" />
+      </geometry>
+      <material
+        name="">
+        <color
+          rgba="0.86667 0.86667 0.8902 1" />
+      </material>
+    </visual>
+    <collision>
+      <origin
+        xyz="0 0 0"
+        rpy="0 0 0" />
+      <geometry>
+        <mesh
+          filename="file://$(find rm_description)/meshes/rm_63_arm/base_link.STL" />
+      </geometry>
+    </collision>
+  </link>
+  <link
+    name="link1">
+    <inertial>
+      <origin
+        xyz="-0.030909 -0.0013023 -0.0053121"
+        rpy="0 0 0" />
+      <mass
+        value="1.7668" />
+      <inertia
+        ixx="0.0014534"
+        ixy="-0.00017578"
+        ixz="0.0002802"
+        iyy="0.0043772"
+        iyz="1.7209E-05"
+        izz="0.0040911" />
+    </inertial>
+    <visual>
+      <origin
+        xyz="0 0 0"
+        rpy="0 0 0" />
+      <geometry>
+        <mesh
+          filename="file://$(find rm_description)/meshes/rm_63_arm/link1.STL" />
+      </geometry>
+      <material
+        name="">
+        <color
+          rgba="1 1 1 1" />
+      </material>
+    </visual>
+    <collision>
+      <origin
+        xyz="0 0 0"
+        rpy="0 0 0" />
+      <geometry>
+        <mesh
+          filename="file://$(find rm_description)/meshes/rm_63_arm/link1.STL" />
+      </geometry>
+    </collision>
+  </link>
+  <joint
+    name="joint1"
+    type="revolute">
+    <origin
+      xyz="0 0 0.172"
+      rpy="0 0 0" />
+    <parent
+      link="base_link" />
+    <child
+      link="link1" />
+    <axis
+      xyz="0 0 1" />
+    <limit
+      lower="-3.107"
+      upper="3.107"
+      effort="100"
+      velocity="1" />
+  </joint>
+  </xacro:if>
+<xacro:if value="${ base_type =='base_link_III' }">
+    <link
+    name="base_link">
+    <inertial>
+      <origin
+        xyz="0.000204933302096124 -8.24661684233942E-05 0.0435919339026087"
+        rpy="0 0 0" />
+      <mass
+        value="0.604237569846431" />
+      <inertia
+        ixx="0.00082415777403083"
+        ixy="2.9270718368632E-06"
+        ixz="-2.8722520476522E-05"
+        iyy="0.000820579526371655"
+        iyz="2.21535061552891E-06"
+        izz="0.000685679517381249" />
+    </inertial>
+    <visual>
+      <origin
+        xyz="0 0 0"
+        rpy="0 0 0" />
+      <geometry>
+        <mesh
+          filename="file://$(find rm_description)/meshes/rm_63_arm/base_link_III.STL" />
+      </geometry>
+      <material
+        name="">
+        <color
+          rgba="0.792156862745098 0.819607843137255 0.933333333333333 1" />
+      </material>
+    </visual>
+    <collision>
+      <origin
+        xyz="0 0 0"
+        rpy="0 0 0" />
+      <geometry>
+        <mesh
+          filename="file://$(find rm_description)/meshes/rm_63_arm/base_link_III.STL" />
+      </geometry>
+    </collision>
+  </link>
+  <link
+    name="link1">
+    <inertial>
+      <origin
+        xyz="-0.030909 -0.0013023 -0.0053121"
+        rpy="0 0 0" />
+      <mass
+        value="1.7668" />
+      <inertia
+        ixx="0.0014534"
+        ixy="-0.00017578"
+        ixz="0.0002802"
+        iyy="0.0043772"
+        iyz="1.7209E-05"
+        izz="0.0040911" />
+    </inertial>
+    <visual>
+      <origin
+        xyz="0 0 0"
+        rpy="0 0 0" />
+      <geometry>
+        <mesh
+          filename="file://$(find rm_description)/meshes/rm_63_arm/link1_III.STL" />
+      </geometry>
+      <material
+        name="">
+        <color
+          rgba="1 1 1 1" />
+      </material>
+    </visual>
+    <collision>
+      <origin
+        xyz="0 0 0"
+        rpy="0 0 0" />
+      <geometry>
+        <mesh
+          filename="file://$(find rm_description)/meshes/rm_63_arm/link1_III.STL" />
+      </geometry>
+    </collision>
+  </link>
+  <joint
+    name="joint1"
+    type="revolute">
+    <origin
+      xyz="0 0 0.1625"
+      rpy="0 0 0" />
+    <parent
+      link="base_link" />
+    <child
+      link="link1" />
+    <axis
+      xyz="0 0 1" />
+    <limit
+      lower="-3.107"
+      upper="3.107"
+      effort="100"
+      velocity="1" />
+  </joint>
+  </xacro:if>
+  <link
+    name="link2">
+    <inertial>
+      <origin
+        xyz="0.16852 9.8217E-07 -0.077258"
+        rpy="0 0 0" />
+      <mass
+        value="4.3415" />
       <inertia
         ixx="0"
@@ -27,5 +229,5 @@
       <geometry>
         <mesh
-          filename="file://$(find rm_description)/meshes/rm_63_arm/base_link.STL" />
+          filename="file://$(find rm_description)/meshes/rm_63_arm/link2.STL" />
       </geometry>
       <material
@@ -41,16 +243,34 @@
       <geometry>
         <mesh
-          filename="file://$(find rm_description)/meshes/rm_63_arm/base_link.STL" />
-      </geometry>
-    </collision>
-  </link>
+          filename="file://$(find rm_description)/meshes/rm_63_arm/link2.STL" />
+      </geometry>
+    </collision>
+  </link>
+  <joint
+    name="joint2"
+    type="revolute">
+    <origin
+      xyz="-0.086 0 0"
+      rpy="-1.5708 -1.5708 0" />
+    <parent
+      link="link1" />
+    <child
+      link="link2" />
+    <axis
+      xyz="0 0 1" />
+    <limit
+      lower="-3.107"
+      upper="3.107"
+      effort="100"
+      velocity="1" />
+  </joint>
   <link
-    name="link1">
-    <inertial>
-      <origin
-        xyz="-0.030909 -0.0013023 -0.0053121"
-        rpy="0 0 0" />
-      <mass
-        value="1.7668" />
+    name="link3">
+    <inertial>
+      <origin
+        xyz="0.034488 -0.010948 -0.0056239"
+        rpy="0 0 0" />
+      <mass
+        value="1.7286" />
       <inertia
         ixx="0"
@@ -67,32 +287,90 @@
       <geometry>
         <mesh
-          filename="file://$(find rm_description)/meshes/rm_63_arm/link1.STL" />
-      </geometry>
-      <material
-        name="">
-        <color
-          rgba="1 1 1 1" />
-      </material>
-    </visual>
-    <collision>
-      <origin
-        xyz="0 0 0"
-        rpy="0 0 0" />
-      <geometry>
-        <mesh
-          filename="file://$(find rm_description)/meshes/rm_63_arm/link1.STL" />
-      </geometry>
-    </collision>
-  </link>
-  <joint
-    name="joint1"
-    type="revolute">
-    <origin
-      xyz="0 0 0.1625"
-      rpy="0 0 0" />
-    <parent
-      link="base_link" />
-    <child
-      link="link1" />
+          filename="file://$(find rm_description)/meshes/rm_63_arm/link3.STL" />
+      </geometry>
+      <material
+        name="">
+        <color
+          rgba="0.86667 0.86667 0.8902 1" />
+      </material>
+    </visual>
+    <collision>
+      <origin
+        xyz="0 0 0"
+        rpy="0 0 0" />
+      <geometry>
+        <mesh
+          filename="file://$(find rm_description)/meshes/rm_63_arm/link3.STL" />
+      </geometry>
+    </collision>
+  </link>
+  <joint
+    name="joint3"
+    type="revolute">
+    <origin
+      xyz="0.38 0 0"
+      rpy="0 0 1.5708" />
+    <parent
+      link="link2" />
+    <child
+      link="link3" />
+    <axis
+      xyz="0 0 1" />
+    <limit
+      lower="-3.107"
+      upper="2.531"
+      effort="100"
+      velocity="1" />
+  </joint>
+  <link
+    name="link4">
+    <inertial>
+      <origin
+        xyz="4.1778E-07 -0.030483 -0.19739"
+        rpy="0 0 0" />
+      <mass
+        value="2.4734" />
+      <inertia
+        ixx="0"
+        ixy="0"
+        ixz="0"
+        iyy="0"
+        iyz="0"
+        izz="0" />i
+    </inertial>
+    <visual>
+      <origin
+        xyz="0 0 0"
+        rpy="0 0 0" />
+      <geometry>
+        <mesh
+          filename="file://$(find rm_description)/meshes/rm_63_arm/link4.STL" />
+      </geometry>
+      <material
+        name="">
+        <color
+          rgba="0.86667 0.86667 0.8902 1" />
+      </material>
+    </visual>
+    <collision>
+      <origin
+        xyz="0 0 0"
+        rpy="0 0 0" />
+      <geometry>
+        <mesh
+          filename="file://$(find rm_description)/meshes/rm_63_arm/link4.STL" />
+      </geometry>
+    </collision>
+  </link>
+  <joint
+    name="joint4"
+    type="revolute">
+    <origin
+      xyz="0.069 -0.405 0"
+      rpy="1.5708 0 0" />
+    <parent
+      link="link3" />
+    <child
+      link="link4" />
     <axis
       xyz="0 0 1" />
@@ -104,11 +382,11 @@
   </joint>
   <link
-    name="link2">
-    <inertial>
-      <origin
-        xyz="0.16852 9.8217E-07 -0.077258"
-        rpy="0 0 0" />
-      <mass
-        value="4.3415" />
+    name="link5">
+    <inertial>
+      <origin
+        xyz="5.2596E-06 0.025125 -0.0072574"
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
File: rm_moveit2_config/rm_63_config/config/rml_63_6fb_description.urdf.xacro (robot description, xacro)
@@ -5,6 +5,8 @@
     <!-- arg->property -->
     <xacro:property name="link6_type" value="$(arg link6_type)" />
+    <xacro:property name="base_type" value="$(arg base_type)" />
     <xacro:include filename="$(find rm_description)/urdf/rml_63.urdf.xacro" >
         link6_type:=$(arg link6_type)
+        base_type:=$(arg base_type)
     </xacro:include>
     <!-- Import control_xacro -->

Commit message: doc:升级ROS21.6.0版本，主要修改项：1添加RML63III型标识，2添加三代modbus接口，3rm_driver doc中添加相关说明，4rm_driver config添加udp相关配置，5部分其他接口。

File: rm_description/urdf/rml_63.urdf (robot description, URDF)
Before this commit: robot rml_63_description, 7 links, 6 joints
Joints:
- joint joint1: origin xyz=0 0 0.1625 rpy=0 0 0 -> xyz=0 0 0.172 rpy=0 0 0

File: rm_description/urdf/rml_63_gazebo.urdf (robot description, URDF)
Before this commit: robot rml_63_description, 7 links, 6 joints
Joints:
- joint joint1: origin xyz=0 0 0.1625 rpy=0 0 0 -> xyz=0 0 0.172 rpy=0 0 0

File: rm_moveit2_config/rm_63_config/config/rml_63_description.urdf.xacro (robot description, xacro)
@@ -5,6 +5,8 @@
     <!-- arg->property -->
     <xacro:property name="link6_type" value="$(arg link6_type)" />
+    <xacro:property name="base_type" value="$(arg base_type)" />
     <xacro:include filename="$(find rm_description)/urdf/rml_63.urdf.xacro" >
         link6_type:=$(arg link6_type)
+        base_type:=$(arg base_type)
     </xacro:include>
     <!-- Import control_xacro -->
