Commit message: 更新全系列机械臂 URDF（算法已校核版本）机器 mesh 文件引用路径~

File: rm_description/urdf/rm_65_6f.urdf (robot description, URDF)
Before this commit: robot rm_65_6f_description, 7 links, 6 joints
Links:
- link Link1: geometry collision mesh filename=package://rm_description/meshes/rm_65_arm/link1.STL; visual mesh filename=package://rm_description/meshes/rm_65_arm/link1.STL
- link Link2: geometry collision mesh filename=package://rm_description/meshes/rm_65_arm/link2.STL; visual mesh filename=package://rm_description/meshes/rm_65_arm/link2.STL
- link Link3: geometry collision mesh filename=package://rm_description/meshes/rm_65_arm/link3.STL; visual mesh filename=package://rm_description/meshes/rm_65_arm/link3.STL
- link Link4: geometry collision mesh filename=package://rm_description/meshes/rm_65_arm/link4.STL; visual mesh filename=package://rm_description/meshes/rm_65_arm/link4.STL
- link Link5: geometry collision mesh filename=package://rm_description/meshes/rm_65_arm/link5.STL; visual mesh filename=package://rm_description/meshes/rm_65_arm/link5.STL
- link Link6: geometry collision mesh filename=package://rm_description/meshes/rm_65_arm/link6_6f.STL; visual mesh filename=package://rm_description/meshes/rm_65_arm/link6_6f.STL
- link base_link: geometry collision mesh filename=package://rm_description/meshes/rm_65_arm/base_link.STL; visual mesh filename=package://rm_description/meshes/rm_65_arm/base_link.STL

File: rm_description/urdf/rm_65_6fb.urdf (robot description, URDF)
Before this commit: robot RM65-6F, 7 links, 6 joints
Links:
- link Link1: geometry collision mesh filename=package://rm_description/meshes/rm_65_arm/link1.STL; visual mesh filename=package://rm_description/meshes/rm_65_arm/link1.STL
- link Link2: geometry collision mesh filename=package://rm_description/meshes/rm_65_arm/link2.STL; visual mesh filename=package://rm_description/meshes/rm_65_arm/link2.STL
- link Link3: geometry collision mesh filename=package://rm_description/meshes/rm_65_arm/link3.STL; visual mesh filename=package://rm_description/meshes/rm_65_arm/link3.STL
- link Link4: geometry collision mesh filename=package://rm_description/meshes/rm_65_arm/link4.STL; visual mesh filename=package://rm_description/meshes/rm_65_arm/link4.STL
- link Link5: geometry collision mesh filename=package://rm_description/meshes/rm_65_arm/link5.STL; visual mesh filename=package://rm_description/meshes/rm_65_arm/link5.STL
- link Link6: geometry collision mesh filename=package://rm_description/meshes/rm_65_arm/link6_6fb.STL; visual mesh filename=package://rm_description/meshes/rm_65_arm/link6_6fb.STL
- link base_link: geometry collision mesh filename=package://rm_description/meshes/rm_65_arm/base_link.STL; visual mesh filename=package://rm_description/meshes/rm_65_arm/base_link.STL

File: rm_description/urdf/rm_75_6f.urdf (robot description, URDF)
Before this commit: robot rm_75_6f_description, 8 links, 7 joints
Links:
- link Link1: geometry collision mesh filename=package://rm_description/meshes/rm_75_arm/link1.STL; visual mesh filename=package://rm_description/meshes/rm_75_arm/link1.STL
- link Link2: geometry collision mesh filename=package://rm_description/meshes/rm_75_arm/link2.STL; visual mesh filename=package://rm_description/meshes/rm_75_arm/link2.STL
- link Link3: geometry collision mesh filename=package://rm_description/meshes/rm_75_arm/link3.STL; visual mesh filename=package://rm_description/meshes/rm_75_arm/link3.STL
- link Link4: geometry collision mesh filename=package://rm_description/meshes/rm_75_arm/link4.STL; visual mesh filename=package://rm_description/meshes/rm_75_arm/link4.STL
- link Link5: geometry collision mesh filename=package://rm_description/meshes/rm_75_arm/link5.STL; visual mesh filename=package://rm_description/meshes/rm_75_arm/link5.STL
- link Link6: geometry collision mesh filename=package://rm_description/meshes/rm_75_arm/link6.STL; visual mesh filename=package://rm_description/meshes/rm_75_arm/link6.STL
- link Link7: geometry collision mesh filename=package://rm_description/meshes/rm_75_arm/link7_6f.STL; visual mesh filename=package://rm_description/meshes/rm_75_arm/link7_6f.STL
- link base_link: geometry collision mesh filename=package://rm_description/meshes/rm_75_arm/base_link.STL; visual mesh filename=package://rm_description/meshes/rm_75_arm/base_link.STL

File: rm_description/urdf/rm_75_6fb.urdf (robot description, URDF)
Before this commit: robot RM75-6F, 8 links, 7 joints
Links:
- link Link7: geometry collision mesh filename=package://rm_description/meshes/rm_75_arm/link7_6fb.STL; visual mesh filename=package://rm_description/meshes/rm_75_arm/link7_6fb.STL
- link Link_1: geometry collision mesh filename=package://rm_description/meshes/rm_75_arm/link1.STL; visual mesh filename=package://rm_description/meshes/rm_75_arm/link1.STL
- link Link_2: geometry collision mesh filename=package://rm_description/meshes/rm_75_arm/link2.STL; visual mesh filename=package://rm_description/meshes/rm_75_arm/link2.STL
- link Link_3: geometry collision mesh filename=package://rm_description/meshes/rm_75_arm/link3.STL; visual mesh filename=package://rm_description/meshes/rm_75_arm/link3.STL
- link Link_4: geometry collision mesh filename=package://rm_description/meshes/rm_75_arm/link4.STL; visual mesh filename=package://rm_description/meshes/rm_75_arm/link4.STL
- link Link_5: geometry collision mesh filename=package://rm_description/meshes/rm_75_arm/link5.STL; visual mesh filename=package://rm_description/meshes/rm_75_arm/link5.STL
- link Link_6: geometry collision mesh filename=package://rm_description/meshes/rm_75_arm/link6.STL; visual mesh filename=package://rm_description/meshes/rm_75_arm/link6.STL
- link base_link: geometry collision mesh filename=package://rm_description/meshes/rm_75_arm/base_link.STL; visual mesh filename=package://rm_description/meshes/rm_75_arm/base_link.STL

File: rm_description/urdf/rm_eco63.urdf (robot description, URDF)
Before this commit: robot rm_eco63, 7 links, 6 joints
Links:
- added link base_root
Joints:
- added joint base_root_joint: type fixed, parent base_root, child base_link, origin xyz=0 0 0 rpy=0 0 0

File: rm_description/urdf/rm_eco63.urdf.xacro (robot description, xacro)
@@ -1,8 +1,15 @@
 <?xml version="1.0" encoding="utf-8"?>
-<robot  name="rm_eco63_description" xmlns:xacro="http://www.ros.org/wiki/xacro">
+<robot  name="rm_eco63" xmlns:xacro="http://www.ros.org/wiki/xacro">
     <!-- link6_type -->
     <xacro:arg name="link6_type" default="Link6" />
     <!-- arg->property -->
     <xacro:property name="link6_type" value="$(arg link6_type)" />
+    <!-- KDL cannot use an inertial root link, so keep base_link under a massless root. -->
+    <link name="base_root" />
+    <joint name="base_root_joint" type="fixed">
+      <origin xyz="0 0 0" rpy="0 0 0" />
+      <parent link="base_root" />
+      <child link="base_link" />
+    </joint>
     <link
     name="base_link">

File: rm_description/urdf/rm_eco63_6fb.urdf (robot description, URDF)
Before this commit: robot ECO63-6FB-URDF, 7 links, 6 joints
Links:
- link Link1: geometry collision mesh filename=file://$(find rm_description)/meshes/rm_eco63_arm/Link1.STL; visual mesh filename=file://$(find rm_description)/meshes/rm_eco63_arm/Link1.STL
- link Link2: geometry collision mesh filename=file://$(find rm_description)/meshes/rm_eco63_arm/Link2.STL; visual mesh filename=file://$(find rm_description)/meshes/rm_eco63_arm/Link2.STL
- link Link3: geometry collision mesh filename=file://$(find rm_description)/meshes/rm_eco63_arm/Link3.STL; visual mesh filename=file://$(find rm_description)/meshes/rm_eco63_arm/Link3.STL
- link Link4: geometry collision mesh filename=file://$(find rm_description)/meshes/rm_eco63_arm/Link4.STL; visual mesh filename=file://$(find rm_description)/meshes/rm_eco63_arm/Link4.STL
- link Link5: geometry collision mesh filename=file://$(find rm_description)/meshes/rm_eco63_arm/Link5.STL; visual mesh filename=file://$(find rm_description)/meshes/rm_eco63_arm/Link5.STL
- link Link6: geometry collision mesh filename=file://$(find rm_description)/meshes/rm_eco63_arm/Link6_6fb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; visual mesh filename=file://$(find rm_description)/meshes/rm_eco63_arm/Link6_6fb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
- link base_link: geometry collision mesh filename=file://$(find rm_description)/meshes/rm_eco63_arm/base_link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; visual mesh filename=file://$(find rm_description)/meshes/rm_eco63_arm/base_link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

File: rm_description/urdf/rm_eco65_6f.urdf (robot description, URDF)
Before this commit: robot eco65, 7 links, 6 joints
Links:
- link Link1: geometry collision mesh filename=package://rm_description/meshes/rm_eco65_arm/Link1.STL; visual mesh filename=package://rm_description/meshes/rm_eco65_arm/Link1.STL
- link Link2: geometry collision mesh filename=package://rm_description/meshes/rm_eco65_arm/Link2.STL; visual mesh filename=package://rm_description/meshes/rm_eco65_arm/Link2.STL
- link Link3: geometry collision mesh filename=package://rm_description/meshes/rm_eco65_arm/Link3.STL; visual mesh filename=package://rm_description/meshes/rm_eco65_arm/Link3.STL
- link Link4: geometry collision mesh filename=package://rm_description/meshes/rm_eco65_arm/Link4.STL; visual mesh filename=package://rm_description/meshes/rm_eco65_arm/Link4.STL
- link Link5: geometry collision mesh filename=package://rm_description/meshes/rm_eco65_arm/Link5.STL; visual mesh filename=package://rm_description/meshes/rm_eco65_arm/Link5.STL
- link Link6: geometry collision mesh filename=package://rm_description/meshes/rm_eco65_arm/Link6_6f.STL; visual mesh filename=package://rm_description/meshes/rm_eco65_arm/Link6_6f.STL
- link baselink: geometry collision mesh filename=package://rm_description/meshes/rm_eco65_arm/baselink.STL; visual mesh filename=package://rm_description/meshes/rm_eco65_arm/baselink.STL

File: rm_description/urdf/rm_eco65_6fb.urdf (robot description, URDF)
Before this commit: robot 0000-eco65_URDF(2), 7 links, 6 joints
Links:
- link base_link: geometry collision mesh filename=package://rm_description/meshes/rm_eco65_arm/baselink.STL; visual mesh filename=package://rm_description/meshes/rm_eco65_arm/baselink.STL
- link link1: geometry collision mesh filename=package://rm_description/meshes/rm_eco65_arm/Link1.STL; visual mesh filename=package://rm_description/meshes/rm_eco65_arm/Link1.STL
- link link2: geometry collision mesh filename=package://rm_description/meshes/rm_eco65_arm/Link2.STL; visual mesh filename=package://rm_description/meshes/rm_eco65_arm/Link2.STL
- link link3: geometry collision mesh filename=package://rm_description/meshes/rm_eco65_arm/Link3.STL; visual mesh filename=package://rm_description/meshes/rm_eco65_arm/Link3.STL
- link link4: geometry collision mesh filename=package://rm_description/meshes/rm_eco65_arm/Link4.STL; visual mesh filename=package://rm_description/meshes/rm_eco65_arm/Link4.STL
- link link5: geometry collision mesh filename=package://rm_description/meshes/rm_eco65_arm/Link5.STL; visual mesh filename=package://rm_description/meshes/rm_eco65_arm/Link5.STL
- link link6: geometry collision mesh filename=package://rm_description/meshes/rm_eco65_arm/Link6_6fb.STL; visual mesh filename=package://rm_description/meshes/rm_eco65_arm/Link6_6fb.STL
