Commit message: V1.7.0

File: rm_description/urdf/rm_rx75-6fb.urdf.xacro (robot description, xacro)
@@ -138,5 +138,5 @@
       <geometry>
         <mesh
-          filename="package://rm_description/meshes/rm_rx75_arm/rm_rx75_left_arm/Link2.STL" />
+          filename="package://rm_description/meshes/rm_rx75_arm/rm_rx75_left_arm/Link2L.STL" />
       </geometry>
       <material
@@ -152,5 +152,5 @@
       <geometry>
         <mesh
-          filename="package://rm_description/meshes/rm_rx75_arm/rm_rx75_left_arm/Link2.STL" />
+          filename="package://rm_description/meshes/rm_rx75_arm/rm_rx75_left_arm/Link2L.STL" />
       </geometry>
     </collision>
@@ -167,8 +167,8 @@
       link="left_Link2" />
     <axis
-      xyz="0 0 -1" />
-    <limit
-      lower="-3.837"
-      upper="0.697"
+      xyz="0 0 1" />
+    <limit
+      lower="-0.697"
+      upper="3.837"
       effort="60"
       velocity="3.14" />

File: rm_description/urdf/rm_rx75-6fb_v.urdf.xacro (robot description, xacro)
@@ -169,6 +169,6 @@
       xyz="0 0 1" />
     <limit
-      lower="-3.837"
-      upper="0.697"
+      lower="-0.697"
+      upper="3.837"
       effort="60"
       velocity="3.14" />

File: rm_gazebo/config/gazebo_eco63_description.urdf.xacro (robot description, xacro)
@@ -1,4 +1,5 @@
 <?xml version="1.0"?>
 <robot xmlns:xacro="http://www.ros.org/wiki/xacro" name="rm_eco63_description">
+    <xacro:arg name="link6_type" default="Link6" />
     <!-- Used for fixing robot to Gazebo 'base_link' 将机械手的基座固定在世界坐标上-->
     <link name="world"/>
@@ -7,6 +8,9 @@
         <child link="base_link"/>
     </joint>
-    <!-- Import claw_description urdf file -->
-    <xacro:include filename="$(find rm_description)/urdf/rm_eco63_gazebo.urdf" />
+    <!-- Import ECO63 robot description. Use the xacro variant so Gazebo gets valid joint limits. -->
+    <xacro:property name="link6_type" value="$(arg link6_type)" />
+    <xacro:include filename="$(find rm_description)/urdf/rm_eco63_gazebo.urdf.xacro" >
+        link6_type:=$(arg link6_type)
+    </xacro:include>
     <!-- 对一些link进行gazebo的属性设置 -->
     <gazebo reference="base_link">

File: rm_gazebo/config/gazebo_rx75_6fb_description.urdf.xacro (robot description, xacro)
@@ -193,5 +193,5 @@
     <gazebo>
         <plugin filename="gz_ros2_control-system" name="gz_ros2_control::GazeboSimROS2ControlPlugin">
-            <parameters>$(find rm_rx75_6fb_config)/config/ros2_controllers.yaml</parameters>
+            <parameters>$(find rm_rx75_config)/config/ros2_controllers.yaml</parameters>
             <robot_param>robot_description</robot_param>
             <robot_param_node>robot_state_publisher</robot_param_node>

File: rm_gazebo/config/gazebo_rx75_6fb_v_description.urdf.xacro (robot description, xacro)
@@ -193,5 +193,5 @@
     <gazebo>
         <plugin filename="gz_ros2_control-system" name="gz_ros2_control::GazeboSimROS2ControlPlugin">
-            <parameters>$(find rm_rx75_6fb_v_config)/config/ros2_controllers.yaml</parameters>
+            <parameters>$(find rm_rx75_config)/config/ros2_controllers.yaml</parameters>
             <robot_param>robot_description</robot_param>
             <robot_param_node>robot_state_publisher</robot_param_node>
