Commit message: Add jazzy branch with ROS2 Jazzy Jalisco support

File: rm_description/urdf/rm_65_gazebo.urdf.xacro (robot description, xacro)
@@ -22,10 +22,10 @@
     </inertial> -->
     <inertia
-        ixx="0"
-        ixy="0"
-        ixz="0"
-        iyy="0"
-        iyz="0"
-        izz="0" />
+        ixx="1e-6"
+        ixy="0"
+        ixz="0"
+        iyy="1e-6"
+        iyz="0"
+        izz="1e-6" />
     </inertial>
     <visual>
@@ -70,10 +70,10 @@
     </inertial> -->
     <inertia
-        ixx="0"
-        ixy="0"
-        ixz="0"
-        iyy="0"
-        iyz="0"
-        izz="0" />
+        ixx="1e-6"
+        ixy="0"
+        ixz="0"
+        iyy="1e-6"
+        iyz="0"
+        izz="1e-6" />
     </inertial>
     <visual>
@@ -136,10 +136,10 @@
     </inertial> -->
     <inertia
-        ixx="0"
-        ixy="0"
-        ixz="0"
-        iyy="0"
-        iyz="0"
-        izz="0" />
+        ixx="1e-6"
+        ixy="0"
+        ixz="0"
+        iyy="1e-6"
+        iyz="0"
+        izz="1e-6" />
     </inertial>
     <visual>
@@ -202,10 +202,10 @@
     </inertial> -->
     <inertia
-        ixx="0"
-        ixy="0"
-        ixz="0"
-        iyy="0"
-        iyz="0"
-        izz="0" />
+        ixx="1e-6"
+        ixy="0"
+        ixz="0"
+        iyy="1e-6"
+        iyz="0"
+        izz="1e-6" />
     </inertial>
     <visual>
@@ -268,10 +268,10 @@
     </inertial>-->
     <inertia
-        ixx="0"
-        ixy="0"
-        ixz="0"
-        iyy="0"
-        iyz="0"
-        izz="0" />
+        ixx="1e-6"
+        ixy="0"
+        ixz="0"
+        iyy="1e-6"
+        iyz="0"
+        izz="1e-6" />
     </inertial>
     <visual>
@@ -334,10 +334,10 @@
     </inertial> -->
     <inertia
-        ixx="0"
-        ixy="0"
-        ixz="0"
-        iyy="0"
-        iyz="0"
-        izz="0" />
+        ixx="1e-6"
+        ixy="0"
+        ixz="0"
+        iyy="1e-6"
+        iyz="0"
+        izz="1e-6" />
     </inertial>
     <visual>
@@ -401,10 +401,10 @@
       </inertial> -->
       <inertia
-        ixx="0"
-        ixy="0"
-        ixz="0"
-        iyy="0"
-        iyz="0"
-        izz="0" />
+        ixx="1e-6"
+        ixy="0"
+        ixz="0"
+        iyy="1e-6"
+        iyz="0"
+        izz="1e-6" />
     </inertial>
       <visual>
@@ -469,10 +469,10 @@
       </inertial> -->
       <inertia
-        ixx="0"
-        ixy="0"
-        ixz="0"
-        iyy="0"
-        iyz="0"
-        izz="0" />
+        ixx="1e-6"
+        ixy="0"
+        ixz="0"
+        iyy="1e-6"
+        iyz="0"
+        izz="1e-6" />
       </inertial>
       <visual>
@@ -537,10 +537,10 @@
       </inertial> -->
       <inertia
-        ixx="0"
-        ixy="0"
-        ixz="0"
-        iyy="0"
-        iyz="0"
-        izz="0" />
+        ixx="1e-6"
+        ixy="0"
+        ixz="0"
+        iyy="1e-6"
+        iyz="0"
+        izz="1e-6" />
       </inertial>
       <visual>

File: rm_description/urdf/rm_eco63_gazebo.urdf.xacro (robot description, xacro)
@@ -14,10 +14,10 @@
         value="8.97974481667473" />
       <inertia
-        ixx="0"
-        ixy="0"
-        ixz="0"
-        iyy="0"
-        iyz="0"
-        izz="0" />
+        ixx="0.862297666639592"
+        ixy="-0.00170110773340804"
+        ixz="0.0134260863948258"
+        iyy="0.853404080505364"
+        iyz="-0.0335323790979435"
+        izz="0.021909948868005" />
     </inertial>
     <visual>
@@ -54,10 +54,10 @@
         value="0.656374618338142" />
       <inertia
-        ixx="0"
-        ixy="0"
-        ixz="0"
-        iyy="0"
-        iyz="0"
-        izz="0" />
+        ixx="0.000538922068295209"
+        ixy="-6.49558484347273E-05"
+        ixz="0.000104084843141859"
+        iyy="0.00162201405585815"
+        iyz="6.13990176963193E-06"
+        izz="0.00151559483136641" />
     </inertial>
     <visual>
@@ -112,10 +112,10 @@
         value="5.26262523683375" />
       <inertia
-        ixx="0"
-        ixy="0"
-        ixz="0"
-        iyy="0"
-        iyz="0"
-        izz="0" />
+        ixx="0.00404170032131906"
+        ixy="-5.65174393111021E-07"
+        ixz="0.00121807022294723"
+        iyy="0.109727764384232"
+        iyz="-2.72124756899763E-09"
+        izz="0.110681578185881" />
     </inertial>
     <visual>
@@ -170,10 +170,10 @@
         value="1.3509329667983" />
       <inertia
-        ixx="0"
-        ixy="0"
-        ixz="0"
-        iyy="0"
-        iyz="0"
-        izz="0" />
+        ixx="0.000796925531981305"
+        ixy="-2.89740446981148E-08"
+        ixz="-0.000607432295339128"
+        iyy="0.0219803140031169"
+        iyz="1.84171394643915E-08"
+        izz="0.022157190260175" />
     </inertial>
     <visual>
@@ -228,10 +228,10 @@
         value="0.733001235394853" />
       <inertia
-        ixx="0"
-        ixy="0"
-        ixz="0"
-        iyy="0"
-        iyz="0"
-        izz="0" />
+        ixx="0.000641256799113762"
+        ixy="7.16323347889126E-09"
+        ixz="-6.76890724051393E-09"
+        iyy="0.000512473473605366"
+        iyz="-0.000109077537111131"
+        izz="0.000460316607732565" />
     </inertial>
     <visual>
@@ -286,10 +286,10 @@
         value="0.911747774463918" />
       <inertia
-        ixx="0"
-        ixy="0"
-        ixz="0"
-        iyy="0"
-        iyz="0"
-        izz="0" />
+        ixx="0.000797250089831515"
+        ixy="-3.0783066224908E-08"
+        ixz="-1.86945083800088E-09"
+        iyy="0.000572176795709541"
+        iyz="-0.000145598908387624"
+        izz="0.000625883738000052" />
     </inertial>
     <visual>
@@ -342,13 +342,13 @@
         xyz="0.000922882083248047 -9.40199566012989E-05 -0.0127047090822767"
         rpy="0 0 0" />
-        <mass
+      <mass
         value="0.065035417997418" />
       <inertia
-        ixx="0"
-        ixy="0"
-        ixz="0"
-        iyy="0"
-        iyz="0"
-        izz="0" />
+        ixx="2.11425102567822E-05"
+        ixy="-2.28752901090794E-08"
+        ixz="-2.56006744332993E-08"
+        iyy="1.81097258369991E-05"
+        iyz="-1.0175060606431E-08"
+        izz="3.19000225583591E-05" />
     </inertial>
     <visual>
@@ -387,5 +387,5 @@
       link="Link6" />
     <axis
-      xyz="0 0 -1" />
+      xyz="0 0 1" />
     <limit
       lower="-6.28"
@@ -405,10 +405,10 @@
         value="0.151764173288042" />
       <inertia
-        ixx="0"
-        ixy="0"
-        ixz="0"
-        iyy="0"
-        iyz="0"
-        izz="0" />
+        ixx="2.11425102567822E-05"
+        ixy="4.33059987978739E-07"
+        ixz="6.85384907695856E-07"
+        iyy="1.81097258369991E-05"
+        iyz="-3.58979113769758E-07"
+        izz="3.19000225583591E-05" />
     </inertial>
     <visual>

File: rm_description/urdf/rm_eco65_gazebo.urdf.xacro (robot description, xacro)
@@ -13,5 +13,5 @@
       <mass
         value="0.61127" />
-      <!-- <inertia
+      <inertia
         ixx="0.00080212"
         ixy="3.0281E-06"
@@ -20,12 +20,4 @@
         iyz="1.9749E-06"
         izz="0.00066167" />
-      </inertial> -->
-      <inertia
-        ixx="0"
-        ixy="0"
-        ixz="0"
-        iyy="0"
-        iyz="0"
-        izz="0" />
     </inertial>
     <visual>
@@ -61,5 +53,5 @@
       <mass
         value="0.74247" />
-      <!-- <inertia
+      <inertia
         ixx="0.00081398"
         ixy="-1.9024E-05"
@@ -68,12 +60,4 @@
         iyz="2.0444E-06"
         izz="0.0015286" />
-    </inertial> -->
-    <inertia
-      ixx="0"
-      ixy="0"
-      ixz="0"
-      iyy="0"
-      iyz="0"
-      izz="0" />
     </inertial>
     <visual>
@@ -127,5 +111,5 @@
       <mass
         value="1.3502" />
-      <!-- <inertia
+      <inertia
         ixx="0.012821"
         ixy="-7.2979E-08"
@@ -134,12 +118,4 @@
         iyz="-0.00033755"
         izz="0.012933" />
-    </inertial> -->
-    <inertia
-      ixx="0"
-      ixy="0"
-      ixz="0"
-      iyy="0"
-      iyz="0"
-      izz="0" />
     </inertial>
     <visual>
@@ -193,5 +169,5 @@
       <mass
         value="1.0422" />
-      <!-- <inertia
+      <inertia
         ixx="0.00084115"
         ixy="-2.2514E-08"
@@ -200,12 +176,4 @@
         iyz="-3.3287E-09"
         izz="0.0092482" />
-    </inertial> -->
-    <inertia
-      ixx="0"
-      ixy="0"
-      ixz="0"
-      iyy="0"
-      iyz="0"
-      izz="0" />
     </inertial>
     <visual>
@@ -259,5 +227,5 @@
       <mass
         value="0.27383" />
-      <!-- <inertia
+      <inertia
         ixx="0.00024751"
         ixy="-5.6849E-09"
@@ -266,12 +234,4 @@
         iyz="-2.8552E-05"
         izz="0.00019295"/>
-    </inertial> -->
-    <inertia
-      ixx="0"
-      ixy="0"
-      ixz="0"
-      iyy="0"
-      iyz="0"
-      izz="0" />
     </inertial>
     <visual>
@@ -325,5 +285,5 @@
       <mass
         value="0.27794" />
-      <!-- <inertia
+      <inertia
         ixx="0.00024751"
         ixy="-5.6849E-09"
@@ -332,12 +292,4 @@
         iyz="-2.8552E-05"
         izz="0.00019295" />
-    </inertial> -->
-    <inertia
-      ixx="0"
-      ixy="0"
-      ixz="0"
-      iyy="0"
-      iyz="0"
-      izz="0" />
     </inertial>
     <visual>
@@ -392,5 +344,5 @@
             <mass
                 value="0.033025" />
-            <!-- <inertia
+            <inertia
                 ixx="1.2968E-05"
                 ixy="-7.8692E-07"
@@ -399,12 +351,4 @@
                 iyz="-1.2002E-07"
                 izz="2.0405E-05" />
-            </inertial> -->
-            <inertia
-              ixx="0"
-              ixy="0"
-              ixz="0"
-              iyy="0"
-              iyz="0"
-              izz="0" />
             </inertial>
             <visual>
@@ -460,5 +404,5 @@
                 <mass
                 value="0.14611108984048" />
-                <!-- <inertia
+                <inertia
                 ixx="7.05928109974802E-05"
                 ixy="-1.19201783223218E-06"
@@ -467,12 +411,4 @@
                 iyz="4.34362652271675E-07"
                 izz="6.18079595264477E-05" />
-            </inertial> -->
-            <inertia
-              ixx="0"
-              ixy="0"
-              ixz="0"
-              iyy="0"
-              iyz="0"
-              izz="0" />
             </inertial>
             <visual>
@@ -482,5 +418,5 @@
                 <geometry>
                 <mesh
-                    filename="file://$(find rm_description)/meshes/rm_eco65_arm/Link6_6f.STL" />
+                    filename="file://$(find rm_description)/meshes/rm_eco65_arm/Link6_6f.STL"/>
                 </geometry>
                 <material
@@ -496,5 +432,5 @@
                 <geometry>
                 <mesh
-                    filename="file://$(find rm_description)/meshes/rm_eco65_arm/Link6_6f.STL "/>
+                    filename="file://$(find rm_description)/meshes/rm_eco65_arm/Link6_6f.STL" />
                 </geometry>
             </collision>
@@ -528,5 +464,5 @@
             <mass
                 value="0.305602477849543" />
-            <!-- <inertia
+            <inertia
                 ixx="0.000113828576086565"
                 ixy="-3.65320556215084E-08"
@@ -535,12 +471,4 @@
                 iyz="-4.34359001412421E-08"
                 izz="0.000126193153799782" />
-            </inertial> -->
-            <inertia
-              ixx="0"
-              ixy="0"
-              ixz="0"
-              iyy="0"
-              iyz="0"
-              izz="0" />
             </inertial>
             <visual>

File: rm_gazebo/config/gazebo_63_6fb_description.urdf.xacro (robot description, xacro)
@@ -1,4 +1,7 @@
 <?xml version="1.0"?>
 <robot xmlns:xacro="http://www.ros.org/wiki/xacro" name="rml_63_description">
+    <xacro:arg name="ros2_control_hardware_plugin" default="gz_ros2_control/GazeboSimSystem"/>
+    <xacro:arg name="ros2_control_plugin_filename" default="gz_ros2_control-system"/>
+    <xacro:arg name="ros2_control_plugin_name" default="gz_ros2_control::GazeboSimROS2ControlPlugin"/>
     <!-- Used for fixing robot to Gazebo 'base_link' 将机械手的基座固定在世界坐标上-->
     <link name="world"/>
@@ -43,11 +46,10 @@
     </gazebo>
     <gazebo>
-        <is_static>true</is_static>
-        <self_collide>true</self_collide>
+                <self_collide>true</self_collide>
     </gazebo>
     <!-- 声明ros2_control -->
     <ros2_control name="GazeboSystem" type="system">
         <hardware>
-            <plugin>gazebo_ros2_control/GazeboSystem</plugin>
+            <plugin>$(arg ros2_control_hardware_plugin)</plugin>
         </hardware>
         <joint name="joint1">
@@ -96,5 +98,5 @@
     <!-- 加载ros2_control插件 -->
     <gazebo>
-        <plugin filename="libgazebo_ros2_control.so" name="gazebo_ros2_control">
+        <plugin filename="$(arg ros2_control_plugin_filename)" name="$(arg ros2_control_plugin_name)">
             <parameters>$(find rm_63_config)/config/ros2_controllers.yaml</parameters>
             <robot_param>robot_description</robot_param>

File: rm_gazebo/config/gazebo_63_III_description.urdf.xacro (robot description, xacro)
@@ -1,4 +1,7 @@
 <?xml version="1.0"?>
 <robot xmlns:xacro="http://www.ros.org/wiki/xacro" name="rml_63_description">
+    <xacro:arg name="ros2_control_hardware_plugin" default="gz_ros2_control/GazeboSimSystem"/>
+    <xacro:arg name="ros2_control_plugin_filename" default="gz_ros2_control-system"/>
+    <xacro:arg name="ros2_control_plugin_name" default="gz_ros2_control::GazeboSimROS2ControlPlugin"/>
     <!-- Used for fixing robot to Gazebo 'base_link' 将机械手的基座固定在世界坐标上-->
     <link name="world"/>
@@ -45,11 +48,10 @@
     </gazebo>
     <gazebo>
-        <is_static>true</is_static>
-        <self_collide>true</self_collide>
+                <self_collide>true</self_collide>
     </gazebo>
     <!-- 声明ros2_control -->
     <ros2_control name="GazeboSystem" type="system">
         <hardware>
-            <plugin>gazebo_ros2_control/GazeboSystem</plugin>
+            <plugin>$(arg ros2_control_hardware_plugin)</plugin>
         </hardware>
         <joint name="joint1">
@@ -98,5 +100,5 @@
     <!-- 加载ros2_control插件 -->
     <gazebo>
-        <plugin filename="libgazebo_ros2_control.so" name="gazebo_ros2_control">
+        <plugin filename="$(arg ros2_control_plugin_filename)" name="$(arg ros2_control_plugin_name)">
             <parameters>$(find rm_63_config)/config/ros2_controllers.yaml</parameters>
             <robot_param>robot_description</robot_param>

File: rm_gazebo/config/gazebo_63_description.urdf.xacro (robot description, xacro)
@@ -1,4 +1,7 @@
 <?xml version="1.0"?>
 <robot xmlns:xacro="http://www.ros.org/wiki/xacro" name="rml_63_description">
+    <xacro:arg name="ros2_control_hardware_plugin" default="gz_ros2_control/GazeboSimSystem"/>
+    <xacro:arg name="ros2_control_plugin_filename" default="gz_ros2_control-system"/>
+    <xacro:arg name="ros2_control_plugin_name" default="gz_ros2_control::GazeboSimROS2ControlPlugin"/>
     <!-- Used for fixing robot to Gazebo 'base_link' 将机械手的基座固定在世界坐标上-->
     <link name="world"/>
@@ -40,11 +43,10 @@
     </gazebo>
     <gazebo>
-        <is_static>true</is_static>
-        <self_collide>true</self_collide>
+                <self_collide>true</self_collide>
     </gazebo>
     <!-- 声明ros2_control -->
     <ros2_control name="GazeboSystem" type="system">
         <hardware>
-            <plugin>gazebo_ros2_control/GazeboSystem</plugin>
+            <plugin>$(arg ros2_control_hardware_plugin)</plugin>
         </hardware>
         <joint name="joint1">
@@ -93,5 +95,5 @@
     <!-- 加载ros2_control插件 -->
     <gazebo>
-        <plugin filename="libgazebo_ros2_control.so" name="gazebo_ros2_control">
+        <plugin filename="$(arg ros2_control_plugin_filename)" name="$(arg ros2_control_plugin_name)">
             <parameters>$(find rm_63_config)/config/ros2_controllers.yaml</parameters>
             <robot_param>robot_description</robot_param>

File: rm_gazebo/config/gazebo_65_6fb_description.urdf.xacro (robot description, xacro)
@@ -1,4 +1,7 @@
 <?xml version="1.0"?>
 <robot xmlns:xacro="http://www.ros.org/wiki/xacro" name="rm_65_description">
+    <xacro:arg name="ros2_control_hardware_plugin" default="gz_ros2_control/GazeboSimSystem"/>
+    <xacro:arg name="ros2_control_plugin_filename" default="gz_ros2_control-system"/>
+    <xacro:arg name="ros2_control_plugin_name" default="gz_ros2_control::GazeboSimROS2ControlPlugin"/>
     <!-- Used for fixing robot to Gazebo 'base_link' 将机械手的基座固定在世界坐标上-->
     <link name="world"/>
@@ -43,11 +46,10 @@
     </gazebo>
     <gazebo>
-        <is_static>true</is_static>
-        <self_collide>true</self_collide>
+                <self_collide>true</self_collide>
     </gazebo>
     <!-- 声明ros2_control -->
     <ros2_control name="GazeboSystem" type="system">
         <hardware>
-            <plugin>gazebo_ros2_control/GazeboSystem</plugin>
+            <plugin>$(arg ros2_control_hardware_plugin)</plugin>
         </hardware>
         <joint name="joint1">
@@ -96,5 +98,5 @@
     <!-- 加载ros2_control插件 -->
     <gazebo>
-        <plugin filename="libgazebo_ros2_control.so" name="gazebo_ros2_control">
+        <plugin filename="$(arg ros2_control_plugin_filename)" name="$(arg ros2_control_plugin_name)">
             <parameters>$(find rm_65_config)/config/ros2_controllers.yaml</parameters>
             <robot_param>robot_description</robot_param>

File: rm_gazebo/config/gazebo_65_description.urdf.xacro (robot description, xacro)
@@ -1,4 +1,7 @@
 <?xml version="1.0"?>
 <robot xmlns:xacro="http://www.ros.org/wiki/xacro" name="rm_65_description">
+    <xacro:arg name="ros2_control_hardware_plugin" default="gz_ros2_control/GazeboSimSystem"/>
+    <xacro:arg name="ros2_control_plugin_filename" default="gz_ros2_control-system"/>
+    <xacro:arg name="ros2_control_plugin_name" default="gz_ros2_control::GazeboSimROS2ControlPlugin"/>
     <!-- Used for fixing robot to Gazebo 'base_link' 将机械手的基座固定在世界坐标上-->
     <link name="world"/>
@@ -40,11 +43,10 @@
     </gazebo>
     <gazebo>
-        <is_static>true</is_static>
-        <self_collide>true</self_collide>
+                <self_collide>true</self_collide>
     </gazebo>
     <!-- 声明ros2_control -->
     <ros2_control name="GazeboSystem" type="system">
         <hardware>
-            <plugin>gazebo_ros2_control/GazeboSystem</plugin>
+            <plugin>$(arg ros2_control_hardware_plugin)</plugin>
         </hardware>
         <joint name="joint1">
@@ -93,5 +95,5 @@
     <!-- 加载ros2_control插件 -->
     <gazebo>
-        <plugin filename="libgazebo_ros2_control.so" name="gazebo_ros2_control">
+        <plugin filename="$(arg ros2_control_plugin_filename)" name="$(arg ros2_control_plugin_name)">
             <parameters>$(find rm_65_config)/config/ros2_controllers.yaml</parameters>
             <robot_param>robot_description</robot_param>

File: rm_gazebo/config/gazebo_75_6fb_description.urdf.xacro (robot description, xacro)
@@ -1,4 +1,7 @@
 <?xml version="1.0"?>
 <robot xmlns:xacro="http://www.ros.org/wiki/xacro" name="rm_75_description">
+    <xacro:arg name="ros2_control_hardware_plugin" default="gz_ros2_control/GazeboSimSystem"/>
+    <xacro:arg name="ros2_control_plugin_filename" default="gz_ros2_control-system"/>
+    <xacro:arg name="ros2_control_plugin_name" default="gz_ros2_control::GazeboSimROS2ControlPlugin"/>
     <!-- Used for fixing robot to Gazebo 'base_link' 将机械手的基座固定在世界坐标上-->
     <link name="world"/>
@@ -47,11 +50,10 @@
     </gazebo>
     <gazebo>
-        <is_static>true</is_static>
-        <self_collide>true</self_collide>
+                <self_collide>true</self_collide>
     </gazebo>
     <!-- 声明ros2_control -->
     <ros2_control name="GazeboSystem" type="system">
         <hardware>
-            <plugin>gazebo_ros2_control/GazeboSystem</plugin>
+            <plugin>$(arg ros2_control_hardware_plugin)</plugin>
         </hardware>
         <joint name="joint1">
@@ -107,5 +109,5 @@
     <!-- 加载ros2_control插件 -->
     <gazebo>
-        <plugin filename="libgazebo_ros2_control.so" name="gazebo_ros2_control">
+        <plugin filename="$(arg ros2_control_plugin_filename)" name="$(arg ros2_control_plugin_name)">
             <parameters>$(find rm_75_config)/config/ros2_controllers.yaml</parameters>
             <robot_param>robot_description</robot_param>

File: rm_gazebo/config/gazebo_75_description.urdf.xacro (robot description, xacro)
@@ -1,4 +1,7 @@
 <?xml version="1.0"?>
 <robot xmlns:xacro="http://www.ros.org/wiki/xacro" name="rm_75_description">
+    <xacro:arg name="ros2_control_hardware_plugin" default="gz_ros2_control/GazeboSimSystem"/>
+    <xacro:arg name="ros2_control_plugin_filename" default="gz_ros2_control-system"/>
+    <xacro:arg name="ros2_control_plugin_name" default="gz_ros2_control::GazeboSimROS2ControlPlugin"/>
     <!-- Used for fixing robot to Gazebo 'base_link' 将机械手的基座固定在世界坐标上-->
     <link name="world"/>
@@ -44,11 +47,10 @@
     </gazebo>
     <gazebo>
-        <is_static>true</is_static>
-        <self_collide>true</self_collide>
+                <self_collide>true</self_collide>
     </gazebo>
     <!-- 声明ros2_control -->
     <ros2_control name="GazeboSystem" type="system">
         <hardware>
-            <plugin>gazebo_ros2_control/GazeboSystem</plugin>
+            <plugin>$(arg ros2_control_hardware_plugin)</plugin>
         </hardware>
         <joint name="joint1">
@@ -104,5 +106,5 @@
     <!-- 加载ros2_control插件 -->
     <gazebo>
-        <plugin filename="libgazebo_ros2_control.so" name="gazebo_ros2_control">
+        <plugin filename="$(arg ros2_control_plugin_filename)" name="$(arg ros2_control_plugin_name)">
             <parameters>$(find rm_75_config)/config/ros2_controllers.yaml</parameters>
             <robot_param>robot_description</robot_param>
