Commit message: Add jazzy branch with ROS2 Jazzy Jalisco support

File: rm_gazebo/config/gazebo_eco63_6fb_description.urdf.xacro (robot description, xacro)
@@ -1,4 +1,7 @@
 <?xml version="1.0"?>
 <robot xmlns:xacro="http://www.ros.org/wiki/xacro" name="rm_eco63_description">
+    <xacro:arg name="ros2_control_hardware_plugin" default="gz_ros2_control/GazeboSimSystem"/>
+    <xacro:arg name="ros2_control_plugin_filename" default="gz_ros2_control-system"/>
+    <xacro:arg name="ros2_control_plugin_name" default="gz_ros2_control::GazeboSimROS2ControlPlugin"/>
     <!-- Used for fixing robot to Gazebo 'base_link' 将机械手的基座固定在世界坐标上-->
     <link name="world"/>
@@ -17,37 +20,36 @@
         <gravity>false</gravity>
     </gazebo>
-    <gazebo reference="link1">
+    <gazebo reference="Link1">
         <material>Gazebo/Purple</material>
         <self_collide>false</self_collide>
         <gravity>false</gravity>
     </gazebo>
-    <gazebo reference="link2">
+    <gazebo reference="Link2">
         <material>Gazebo/Red</material>
         <gravity>false</gravity>
     </gazebo>
-    <gazebo reference="link3">
+    <gazebo reference="Link3">
         <material>Gazebo/Blue</material>
         <gravity>false</gravity>
     </gazebo>
-    <gazebo reference="link4">
+    <gazebo reference="Link4">
         <material>Gazebo/Green</material>
         <gravity>false</gravity>
     </gazebo>
-    <gazebo reference="link5">
+    <gazebo reference="Link5">
         <material>Gazebo/Yellow</material>
         <gravity>false</gravity>
     </gazebo>
-    <gazebo reference="link6">
+    <gazebo reference="Link6">
         <material>Gazebo/Orange</material>
         <gravity>false</gravity>
     </gazebo>
     <gazebo>
-        <is_static>true</is_static>
-        <self_collide>true</self_collide>
+                <self_collide>true</self_collide>
     </gazebo>
     <!-- 声明ros2_control -->
     <ros2_control name="GazeboSystem" type="system">
         <hardware>
-            <plugin>gazebo_ros2_control/GazeboSystem</plugin>
+            <plugin>$(arg ros2_control_hardware_plugin)</plugin>
         </hardware>
         <joint name="joint1">
@@ -96,5 +98,5 @@
     <!-- 加载ros2_control插件 -->
     <gazebo>
-        <plugin filename="libgazebo_ros2_control.so" name="gazebo_ros2_control">
+        <plugin filename="$(arg ros2_control_plugin_filename)" name="$(arg ros2_control_plugin_name)">
             <parameters>$(find rm_eco63_config)/config/ros2_controllers.yaml</parameters>
             <robot_param>robot_description</robot_param>

File: rm_gazebo/config/gazebo_eco63_description.urdf.xacro (robot description, xacro)
@@ -1,4 +1,7 @@
 <?xml version="1.0"?>
 <robot xmlns:xacro="http://www.ros.org/wiki/xacro" name="rm_eco63_description">
+    <xacro:arg name="ros2_control_hardware_plugin" default="gz_ros2_control/GazeboSimSystem"/>
+    <xacro:arg name="ros2_control_plugin_filename" default="gz_ros2_control-system"/>
+    <xacro:arg name="ros2_control_plugin_name" default="gz_ros2_control::GazeboSimROS2ControlPlugin"/>
     <!-- Used for fixing robot to Gazebo 'base_link' 将机械手的基座固定在世界坐标上-->
     <link name="world"/>
@@ -8,5 +11,5 @@
     </joint>
     <!-- Import claw_description urdf file -->
-    <xacro:include filename="$(find rm_description)/urdf/rm_eco63_gazebo.urdf" />
+    <xacro:include filename="$(find rm_description)/urdf/rm_eco63_gazebo.urdf.xacro" />
     <!-- 对一些link进行gazebo的属性设置 -->
     <gazebo reference="base_link">
@@ -14,37 +17,36 @@
         <gravity>false</gravity>
     </gazebo>
-    <gazebo reference="link1">
+    <gazebo reference="Link1">
         <material>Gazebo/Purple</material>
         <self_collide>false</self_collide>
         <gravity>false</gravity>
     </gazebo>
-    <gazebo reference="link2">
+    <gazebo reference="Link2">
         <material>Gazebo/Red</material>
         <gravity>false</gravity>
     </gazebo>
-    <gazebo reference="link3">
+    <gazebo reference="Link3">
         <material>Gazebo/Blue</material>
         <gravity>false</gravity>
     </gazebo>
-    <gazebo reference="link4">
+    <gazebo reference="Link4">
         <material>Gazebo/Green</material>
         <gravity>false</gravity>
     </gazebo>
-    <gazebo reference="link5">
+    <gazebo reference="Link5">
         <material>Gazebo/Yellow</material>
         <gravity>false</gravity>
     </gazebo>
-    <gazebo reference="link6">
+    <gazebo reference="Link6">
         <material>Gazebo/Orange</material>
         <gravity>false</gravity>
     </gazebo>
     <gazebo>
-        <is_static>true</is_static>
-        <self_collide>true</self_collide>
+                <self_collide>true</self_collide>
     </gazebo>
     <!-- 声明ros2_control -->
     <ros2_control name="GazeboSystem" type="system">
         <hardware>
-            <plugin>gazebo_ros2_control/GazeboSystem</plugin>
+            <plugin>$(arg ros2_control_hardware_plugin)</plugin>
         </hardware>
         <joint name="joint1">
@@ -93,5 +95,5 @@
     <!-- 加载ros2_control插件 -->
     <gazebo>
-        <plugin filename="libgazebo_ros2_control.so" name="gazebo_ros2_control">
+        <plugin filename="$(arg ros2_control_plugin_filename)" name="$(arg ros2_control_plugin_name)">
             <parameters>$(find rm_eco63_config)/config/ros2_controllers.yaml</parameters>
             <robot_param>robot_description</robot_param>

File: rm_gazebo/config/gazebo_eco65_6fb_description.urdf.xacro (robot description, xacro)
@@ -1,4 +1,7 @@
 <?xml version="1.0"?>
 <robot xmlns:xacro="http://www.ros.org/wiki/xacro" name="rm_eco65_description">
+    <xacro:arg name="ros2_control_hardware_plugin" default="gz_ros2_control/GazeboSimSystem"/>
+    <xacro:arg name="ros2_control_plugin_filename" default="gz_ros2_control-system"/>
+    <xacro:arg name="ros2_control_plugin_name" default="gz_ros2_control::GazeboSimROS2ControlPlugin"/>
     <!-- Used for fixing robot to Gazebo 'base_link' 将机械手的基座固定在世界坐标上-->
     <link name="world"/>
@@ -17,37 +20,36 @@
         <gravity>false</gravity>
     </gazebo>
-    <gazebo reference="link1">
+    <gazebo reference="Link1">
         <material>Gazebo/Purple</material>
         <self_collide>false</self_collide>
         <gravity>false</gravity>
     </gazebo>
-    <gazebo reference="link2">
+    <gazebo reference="Link2">
         <material>Gazebo/Red</material>
         <gravity>false</gravity>
     </gazebo>
-    <gazebo reference="link3">
+    <gazebo reference="Link3">
         <material>Gazebo/Blue</material>
         <gravity>false</gravity>
     </gazebo>
-    <gazebo reference="link4">
+    <gazebo reference="Link4">
         <material>Gazebo/Green</material>
         <gravity>false</gravity>
     </gazebo>
-    <gazebo reference="link5">
+    <gazebo reference="Link5">
         <material>Gazebo/Yellow</material>
         <gravity>false</gravity>
     </gazebo>
-    <gazebo reference="link6">
+    <gazebo reference="Link6">
         <material>Gazebo/Orange</material>
         <gravity>false</gravity>
     </gazebo>
     <gazebo>
-        <is_static>true</is_static>
-        <self_collide>true</self_collide>
+                <self_collide>true</self_collide>
     </gazebo>
     <!-- 声明ros2_control -->
     <ros2_control name="GazeboSystem" type="system">
         <hardware>
-            <plugin>gazebo_ros2_control/GazeboSystem</plugin>
+            <plugin>$(arg ros2_control_hardware_plugin)</plugin>
         </hardware>
         <joint name="joint1">
@@ -96,5 +98,5 @@
     <!-- 加载ros2_control插件 -->
     <gazebo>
-        <plugin filename="libgazebo_ros2_control.so" name="gazebo_ros2_control">
+        <plugin filename="$(arg ros2_control_plugin_filename)" name="$(arg ros2_control_plugin_name)">
             <parameters>$(find rm_eco65_config)/config/ros2_controllers.yaml</parameters>
             <robot_param>robot_description</robot_param>

File: rm_gazebo/config/gazebo_eco65_description.urdf.xacro (robot description, xacro)
@@ -1,4 +1,7 @@
 <?xml version="1.0"?>
 <robot xmlns:xacro="http://www.ros.org/wiki/xacro" name="rm_eco65_description">
+    <xacro:arg name="ros2_control_hardware_plugin" default="gz_ros2_control/GazeboSimSystem"/>
+    <xacro:arg name="ros2_control_plugin_filename" default="gz_ros2_control-system"/>
+    <xacro:arg name="ros2_control_plugin_name" default="gz_ros2_control::GazeboSimROS2ControlPlugin"/>
     <!-- Used for fixing robot to Gazebo 'base_link' 将机械手的基座固定在世界坐标上-->
     <link name="world"/>
@@ -8,5 +11,5 @@
     </joint>
     <!-- Import claw_description urdf file -->
-    <xacro:include filename="$(find rm_description)/urdf/rm_eco65_gazebo.urdf" />
+    <xacro:include filename="$(find rm_description)/urdf/rm_eco65_gazebo.urdf.xacro" />
     <!-- 对一些link进行gazebo的属性设置 -->
     <gazebo reference="baselink">
@@ -14,37 +17,36 @@
         <gravity>false</gravity>
     </gazebo>
-    <gazebo reference="link1">
+    <gazebo reference="Link1">
         <material>Gazebo/Purple</material>
         <self_collide>false</self_collide>
         <gravity>false</gravity>
     </gazebo>
-    <gazebo reference="link2">
+    <gazebo reference="Link2">
         <material>Gazebo/Red</material>
         <gravity>false</gravity>
     </gazebo>
-    <gazebo reference="link3">
+    <gazebo reference="Link3">
         <material>Gazebo/Blue</material>
         <gravity>false</gravity>
     </gazebo>
-    <gazebo reference="link4">
+    <gazebo reference="Link4">
         <material>Gazebo/Green</material>
         <gravity>false</gravity>
     </gazebo>
-    <gazebo reference="link5">
+    <gazebo reference="Link5">
         <material>Gazebo/Yellow</material>
         <gravity>false</gravity>
     </gazebo>
-    <gazebo reference="link6">
+    <gazebo reference="Link6">
         <material>Gazebo/Orange</material>
         <gravity>false</gravity>
     </gazebo>
     <gazebo>
-        <is_static>true</is_static>
-        <self_collide>true</self_collide>
+                <self_collide>true</self_collide>
     </gazebo>
     <!-- 声明ros2_control -->
     <ros2_control name="GazeboSystem" type="system">
         <hardware>
-            <plugin>gazebo_ros2_control/GazeboSystem</plugin>
+            <plugin>$(arg ros2_control_hardware_plugin)</plugin>
         </hardware>
         <joint name="joint1">
@@ -93,5 +95,5 @@
     <!-- 加载ros2_control插件 -->
     <gazebo>
-        <plugin filename="libgazebo_ros2_control.so" name="gazebo_ros2_control">
+        <plugin filename="$(arg ros2_control_plugin_filename)" name="$(arg ros2_control_plugin_name)">
             <parameters>$(find rm_eco65_config)/config/ros2_controllers.yaml</parameters>
             <robot_param>robot_description</robot_param>

File: rm_gazebo/config/gazebo_gen72_II_description.urdf.xacro (robot description, xacro)
@@ -1,4 +1,7 @@
 <?xml version="1.0"?>
 <robot xmlns:xacro="http://www.ros.org/wiki/xacro" name="rm_gen72_description">
+    <xacro:arg name="ros2_control_hardware_plugin" default="gz_ros2_control/GazeboSimSystem"/>
+    <xacro:arg name="ros2_control_plugin_filename" default="gz_ros2_control-system"/>
+    <xacro:arg name="ros2_control_plugin_name" default="gz_ros2_control::GazeboSimROS2ControlPlugin"/>
     <!-- Used for fixing robot to Gazebo 'base_link' 将机械手的基座固定在世界坐标上-->
     <link name="world"/>
@@ -44,11 +47,10 @@
     </gazebo>
     <gazebo>
-        <is_static>true</is_static>
-        <self_collide>true</self_collide>
+                <self_collide>true</self_collide>
     </gazebo>
     <!-- 声明ros2_control -->
     <ros2_control name="GazeboSystem" type="system">
         <hardware>
-            <plugin>gazebo_ros2_control/GazeboSystem</plugin>
+            <plugin>$(arg ros2_control_hardware_plugin)</plugin>
         </hardware>
         <joint name="joint1">
@@ -104,5 +106,5 @@
     <!-- 加载ros2_control插件 -->
     <gazebo>
-        <plugin filename="libgazebo_ros2_control.so" name="gazebo_ros2_control">
+        <plugin filename="$(arg ros2_control_plugin_filename)" name="$(arg ros2_control_plugin_name)">
             <parameters>$(find rm_gen72_config)/config/ros2_controllers.yaml</parameters>
             <robot_param>robot_description</robot_param>

File: rm_gazebo/config/gazebo_gen72_description.urdf.xacro (robot description, xacro)
@@ -1,4 +1,7 @@
 <?xml version="1.0"?>
 <robot xmlns:xacro="http://www.ros.org/wiki/xacro" name="rm_gen72_description">
+    <xacro:arg name="ros2_control_hardware_plugin" default="gz_ros2_control/GazeboSimSystem"/>
+    <xacro:arg name="ros2_control_plugin_filename" default="gz_ros2_control-system"/>
+    <xacro:arg name="ros2_control_plugin_name" default="gz_ros2_control::GazeboSimROS2ControlPlugin"/>
     <!-- Used for fixing robot to Gazebo 'base_link' 将机械手的基座固定在世界坐标上-->
     <link name="world"/>
@@ -44,11 +47,10 @@
     </gazebo>
     <gazebo>
-        <is_static>true</is_static>
-        <self_collide>true</self_collide>
+                <self_collide>true</self_collide>
     </gazebo>
     <!-- 声明ros2_control -->
     <ros2_control name="GazeboSystem" type="system">
         <hardware>
-            <plugin>gazebo_ros2_control/GazeboSystem</plugin>
+            <plugin>$(arg ros2_control_hardware_plugin)</plugin>
         </hardware>
         <joint name="joint1">
@@ -104,5 +106,5 @@
     <!-- 加载ros2_control插件 -->
     <gazebo>
-        <plugin filename="libgazebo_ros2_control.so" name="gazebo_ros2_control">
+        <plugin filename="$(arg ros2_control_plugin_filename)" name="$(arg ros2_control_plugin_name)">
             <parameters>$(find rm_gen72_config)/config/ros2_controllers.yaml</parameters>
             <robot_param>robot_description</robot_param>

File: rm_moveit2_config/rm_63_config/config/rml_63_description.ros2_control.xacro (robot description, xacro)
@@ -2,5 +2,5 @@
 <robot xmlns:xacro="http://www.ros.org/wiki/xacro">
     <xacro:macro name="rml_63_description_ros2_control" params="name initial_positions_file">
-        <xacro:property name="initial_positions" value="${load_yaml(initial_positions_file)['initial_positions']}"/>
+        <xacro:property name="initial_positions" value="${xacro.load_yaml(initial_positions_file)['initial_positions']}"/>
         <ros2_control name="${name}" type="system">
             <hardware>

File: rm_moveit2_config/rm_65_config/config/rm_65_description.ros2_control.xacro (robot description, xacro)
@@ -2,5 +2,5 @@
 <robot xmlns:xacro="http://www.ros.org/wiki/xacro">
     <xacro:macro name="rm_65_description_ros2_control" params="name initial_positions_file">
-        <xacro:property name="initial_positions" value="${load_yaml(initial_positions_file)['initial_positions']}"/>
+        <xacro:property name="initial_positions" value="${xacro.load_yaml(initial_positions_file)['initial_positions']}"/>
         <ros2_control name="${name}" type="system">
             <hardware>

File: rm_moveit2_config/rm_75_config/config/rm_75_description.ros2_control.xacro (robot description, xacro)
@@ -2,5 +2,5 @@
 <robot xmlns:xacro="http://www.ros.org/wiki/xacro">
     <xacro:macro name="rm_75_description_ros2_control" params="name initial_positions_file">
-        <xacro:property name="initial_positions" value="${load_yaml(initial_positions_file)['initial_positions']}"/>
+        <xacro:property name="initial_positions" value="${xacro.load_yaml(initial_positions_file)['initial_positions']}"/>
         <ros2_control name="${name}" type="system">
             <hardware>

File: rm_moveit2_config/rm_eco63_config/config/rm_eco63_description.ros2_control.xacro (robot description, xacro)
@@ -2,5 +2,5 @@
 <robot xmlns:xacro="http://www.ros.org/wiki/xacro">
     <xacro:macro name="rm_eco63_description_ros2_control" params="name initial_positions_file">
-        <xacro:property name="initial_positions" value="${load_yaml(initial_positions_file)['initial_positions']}"/>
+        <xacro:property name="initial_positions" value="${xacro.load_yaml(initial_positions_file)['initial_positions']}"/>
         <ros2_control name="${name}" type="system">
             <hardware>
