Commit message: Add foxy-yifei branch with ROS2 Foxy support

File: rm_description/urdf/rm_eco63.urdf (robot description, URDF)
Before this commit: robot rm_eco63, 7 links, 6 joints
Links:
- added link base_root
Joints:
- added joint base_root_joint: type fixed, parent base_root, child base_link, origin xyz=0 0 0 rpy=0 0 0

File: rm_description/urdf/rm_eco63.urdf.xacro (robot description, xacro)
@@ -1,8 +1,15 @@
 <?xml version="1.0" encoding="utf-8"?>
-<robot  name="rm_eco63_description" xmlns:xacro="http://www.ros.org/wiki/xacro">
+<robot  name="rm_eco63" xmlns:xacro="http://www.ros.org/wiki/xacro">
     <!-- link6_type -->
     <xacro:arg name="link6_type" default="Link6" />
     <!-- arg->property -->
     <xacro:property name="link6_type" value="$(arg link6_type)" />
+    <!-- KDL cannot use an inertial root link, so keep base_link under a massless root. -->
+    <link name="base_root" />
+    <joint name="base_root_joint" type="fixed">
+      <origin xyz="0 0 0" rpy="0 0 0" />
+      <parent link="base_root" />
+      <child link="base_link" />
+    </joint>
     <link
     name="base_link">
@@ -87,5 +94,5 @@
   <joint
     name="joint1"
-    type="revolute">
+    type="continuous">
     <origin
       xyz="0 0 0.1625"
@@ -98,6 +105,4 @@
       xyz="0 0 1" />
     <limit
-      lower="-3.105"
-      upper="3.105"
       effort="60"
       velocity="3.14" />
@@ -261,5 +266,5 @@
   <joint
     name="joint4"
-    type="revolute">
+    type="continuous">
     <origin
       xyz="0.38049 0 -0.054981"
@@ -272,6 +277,4 @@
       xyz="0 0 1" />
     <limit
-      lower="-3.105"
-      upper="3.105"
       effort="10"
       velocity="3.14" />
@@ -319,5 +322,5 @@
   <joint
     name="joint5"
-    type="revolute">
+    type="continuous">
     <origin
       xyz="0 -0.11 -0.0006"
@@ -330,6 +333,4 @@
       xyz="0 0 1" />
     <limit
-      lower="-3.105"
-      upper="3.105"
       effort="10"
       velocity="3.14" />
@@ -378,5 +379,5 @@
   <joint
     name="joint6"
-    type="revolute">
+    type="continuous">
     <origin
       xyz="-0.00010641 0.0797 -0.00010731"
@@ -389,6 +390,4 @@
       xyz="0 0 1" />
     <limit
-      lower="-6.28"
-      upper="6.28"
       effort="10"
       velocity="3.14" />
@@ -438,5 +437,5 @@
   <joint
     name="joint6"
-    type="revolute">
+    type="continuous">
     <origin
       xyz="0 0.0967 0"
@@ -449,6 +448,4 @@
       xyz="0 0 1" />
     <limit
-      lower="-6.28"
-      upper="6.28"
       effort="10"
       velocity="3.14" />

File: rm_gazebo/config/gazebo_63_6fb_description.urdf.xacro (robot description, xacro)
@@ -43,6 +43,5 @@
     </gazebo>
     <gazebo>
-        <is_static>true</is_static>
-        <self_collide>true</self_collide>
+                <self_collide>true</self_collide>
     </gazebo>
     <!-- 声明ros2_control -->

File: rm_gazebo/config/gazebo_63_III_description.urdf.xacro (robot description, xacro)
@@ -45,6 +45,5 @@
     </gazebo>
     <gazebo>
-        <is_static>true</is_static>
-        <self_collide>true</self_collide>
+                <self_collide>true</self_collide>
     </gazebo>
     <!-- 声明ros2_control -->

File: rm_gazebo/config/gazebo_63_description.urdf.xacro (robot description, xacro)
@@ -40,6 +40,5 @@
     </gazebo>
     <gazebo>
-        <is_static>true</is_static>
-        <self_collide>true</self_collide>
+                <self_collide>true</self_collide>
     </gazebo>
     <!-- 声明ros2_control -->

File: rm_gazebo/config/gazebo_65_6fb_description.urdf.xacro (robot description, xacro)
@@ -43,6 +43,5 @@
     </gazebo>
     <gazebo>
-        <is_static>true</is_static>
-        <self_collide>true</self_collide>
+                <self_collide>true</self_collide>
     </gazebo>
     <!-- 声明ros2_control -->

File: rm_gazebo/config/gazebo_65_description.urdf.xacro (robot description, xacro)
@@ -40,6 +40,5 @@
     </gazebo>
     <gazebo>
-        <is_static>true</is_static>
-        <self_collide>true</self_collide>
+                <self_collide>true</self_collide>
     </gazebo>
     <!-- 声明ros2_control -->

File: rm_gazebo/config/gazebo_75_6fb_description.urdf.xacro (robot description, xacro)
@@ -47,6 +47,5 @@
     </gazebo>
     <gazebo>
-        <is_static>true</is_static>
-        <self_collide>true</self_collide>
+                <self_collide>true</self_collide>
     </gazebo>
     <!-- 声明ros2_control -->

File: rm_gazebo/config/gazebo_75_description.urdf.xacro (robot description, xacro)
@@ -44,6 +44,5 @@
     </gazebo>
     <gazebo>
-        <is_static>true</is_static>
-        <self_collide>true</self_collide>
+                <self_collide>true</self_collide>
     </gazebo>
     <!-- 声明ros2_control -->

File: rm_gazebo/config/gazebo_eco63_6fb_description.urdf.xacro (robot description, xacro)
@@ -43,6 +43,5 @@
     </gazebo>
     <gazebo>
-        <is_static>true</is_static>
-        <self_collide>true</self_collide>
+                <self_collide>true</self_collide>
     </gazebo>
     <!-- 声明ros2_control -->

File: rm_gazebo/config/gazebo_eco63_description.urdf.xacro (robot description, xacro)
@@ -1,4 +1,5 @@
 <?xml version="1.0"?>
 <robot xmlns:xacro="http://www.ros.org/wiki/xacro" name="rm_eco63_description">
+    <xacro:arg name="link6_type" default="Link6" />
     <!-- Used for fixing robot to Gazebo 'base_link' 将机械手的基座固定在世界坐标上-->
     <link name="world"/>
@@ -7,6 +8,9 @@
         <child link="base_link"/>
     </joint>
-    <!-- Import claw_description urdf file -->
-    <xacro:include filename="$(find rm_description)/urdf/rm_eco63_gazebo.urdf" />
+    <!-- Import ECO63 robot description. Use the xacro variant so Gazebo gets valid joint limits. -->
+    <xacro:property name="link6_type" value="$(arg link6_type)" />
+    <xacro:include filename="$(find rm_description)/urdf/rm_eco63_gazebo.urdf.xacro" >
+        link6_type:=$(arg link6_type)
+    </xacro:include>
     <!-- 对一些link进行gazebo的属性设置 -->
     <gazebo reference="base_link">
@@ -40,6 +44,5 @@
     </gazebo>
     <gazebo>
-        <is_static>true</is_static>
-        <self_collide>true</self_collide>
+                <self_collide>true</self_collide>
     </gazebo>
     <!-- 声明ros2_control -->

File: rm_gazebo/config/gazebo_eco65_6fb_description.urdf.xacro (robot description, xacro)
@@ -43,6 +43,5 @@
     </gazebo>
     <gazebo>
-        <is_static>true</is_static>
-        <self_collide>true</self_collide>
+                <self_collide>true</self_collide>
     </gazebo>
     <!-- 声明ros2_control -->

File: rm_gazebo/config/gazebo_eco65_description.urdf.xacro (robot description, xacro)
@@ -40,6 +40,5 @@
     </gazebo>
     <gazebo>
-        <is_static>true</is_static>
-        <self_collide>true</self_collide>
+                <self_collide>true</self_collide>
     </gazebo>
     <!-- 声明ros2_control -->

File: rm_gazebo/config/gazebo_gen72_II_description.urdf.xacro (robot description, xacro)
@@ -44,6 +44,5 @@
     </gazebo>
     <gazebo>
-        <is_static>true</is_static>
-        <self_collide>true</self_collide>
+                <self_collide>true</self_collide>
     </gazebo>
     <!-- 声明ros2_control -->

File: rm_gazebo/config/gazebo_gen72_description.urdf.xacro (robot description, xacro)
@@ -44,6 +44,5 @@
     </gazebo>
     <gazebo>
-        <is_static>true</is_static>
-        <self_collide>true</self_collide>
+                <self_collide>true</self_collide>
     </gazebo>
     <!-- 声明ros2_control -->

File: rm_moveit2_config/rm_63_config/config/rml_63_description.ros2_control.xacro (robot description, xacro)
@@ -6,5 +6,5 @@
             <hardware>
                 <!-- By default, set up controllers for simulation. This won't work on real hardware -->
-                <plugin>mock_components/GenericSystem</plugin>
+                <plugin>fake_components/GenericSystem</plugin>
             </hardware>
             <joint name="joint1">

File: rm_moveit2_config/rm_63_config/config/rml_63_description.urdf.xacro (robot description, xacro)
@@ -2,6 +2,12 @@
 <robot xmlns:xacro="http://www.ros.org/wiki/xacro" name="rml_63_description">
     <xacro:arg name="initial_positions_file" default="initial_positions.yaml" />
-    <!-- Import rml_63_description urdf file -->
-    <xacro:include filename="$(find rm_description)/urdf/rml_63.urdf" />
+    <!-- Import rm_65_description urdf file -->
+    <!-- arg->property -->
+    <xacro:property name="link6_type" value="$(arg link6_type)" />
+    <xacro:property name="base_type" value="$(arg base_type)" />
+    <xacro:include filename="$(find rm_description)/urdf/rml_63.urdf.xacro" >
+        link6_type:=$(arg link6_type)
+        base_type:=$(arg base_type)
+    </xacro:include>
     <!-- Import control_xacro -->
     <xacro:include filename="rml_63_description.ros2_control.xacro" />

File: rm_moveit2_config/rm_65_config/config/rm_65_description.ros2_control.xacro (robot description, xacro)
@@ -6,5 +6,5 @@
             <hardware>
                 <!-- By default, set up controllers for simulation. This won't work on real hardware -->
-                <plugin>mock_components/GenericSystem</plugin>
+                <plugin>fake_components/GenericSystem</plugin>
             </hardware>
             <joint name="joint1">

File: rm_moveit2_config/rm_65_config/config/rm_65_description.urdf.xacro (robot description, xacro)
@@ -2,6 +2,10 @@
 <robot xmlns:xacro="http://www.ros.org/wiki/xacro" name="rm_65_description">
     <xacro:arg name="initial_positions_file" default="initial_positions.yaml" />
+    <!-- arg->property -->
+    <xacro:property name="link6_type" value="$(arg link6_type)" />
     <!-- Import rm_65_description urdf file -->
-    <xacro:include filename="$(find rm_description)/urdf/rm_65.urdf" />
+    <xacro:include filename="$(find rm_description)/urdf/rm_65.urdf.xacro" >
+        link6_type:=$(arg link6_type)
+    </xacro:include>
     <!-- Import control_xacro -->
     <xacro:include filename="rm_65_description.ros2_control.xacro" />

File: rm_moveit2_config/rm_75_config/config/rm_75_description.ros2_control.xacro (robot description, xacro)
@@ -6,5 +6,5 @@
             <hardware>
                 <!-- By default, set up controllers for simulation. This won't work on real hardware -->
-                <plugin>mock_components/GenericSystem</plugin>
+                <plugin>fake_components/GenericSystem</plugin>
             </hardware>
             <joint name="joint1">
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
Commit message: Update code from foxy directory

File: rm_description/urdf/rm_eco63.urdf (robot description, URDF)
Before this commit: robot rm_eco63, 8 links, 7 joints
Links:
- link Link1: mass 1.6026 -> 0.656374618338142
- link Link2: mass 2.8169 -> 5.26262523683375
- link Link3: mass 2.6857 -> 1.3509329667983
- link Link4: mass 0.625 -> 0.733001235394853
- link Link5: mass 0.6743 -> 0.911747774463918
- link Link6: mass 0.248 -> 0.065035417997418
- link base_link: mass 1 -> 8.97974481667473
