Commit message: Sync URDF mass/inertia parameters from rm_models

File: rm_description/urdf/rm_65.urdf (robot description, URDF)
Before this commit: robot rm_65_description, 7 links, 6 joints
Links:
- link Link1: mass 0.593563443690403 -> 1.51
- link Link2: mass 0.864175046869043 -> 1.653
- link Link3: mass 0.289633681624654 -> 0.726
- link Link4: mass 0.239419768320061 -> 0.671
- link Link5: mass 0.218799761431678 -> 0.647
- link Link6: mass 0.0649018034311231 -> 0.104
- link base_link: mass 0.841070778135659 -> 1.862

File: rm_description/urdf/rm_65_6f.urdf (robot description, URDF)
Before this commit: robot rm_65_6f_description, 7 links, 6 joints
Links:
- link Link1: mass 0.59356 -> 1.51
- link Link2: mass 0.86418 -> 1.653
- link Link3: mass 0.28963 -> 0.726
- link Link4: mass 0.23941 -> 0.671
- link Link5: mass 0.21879 -> 0.647
- link Link6: mass 0.14433 -> 0.14434
- link base_link: mass 0.84105 -> 1.862

File: rm_description/urdf/rm_65_6fb.urdf (robot description, URDF)
Before this commit: robot RM65-6F, 7 links, 6 joints
Links:
- link Link1: mass 0.593542243994357 -> 1.51
- link Link2: mass 0.86417584142394 -> 1.653
- link Link3: mass 0.289643824525119 -> 0.726
- link Link4: mass 0.239430992940448 -> 0.671
- link Link5: mass 0.21879527056675 -> 0.647
- link Link6: mass 3.04449097371379 -> 0.14434
- link base_link: mass 0.838885281114303 -> 1.862

File: rm_description/urdf/rm_75.urdf (robot description, URDF)
Before this commit: robot rm_75_description, 8 links, 7 joints
Links:
- link Link1: mass 0.593563458735581 -> 1.574
- link Link2: mass 0.432849770310974 -> 1.217
- link Link3: mass 0.431325495678459 -> 1.11
- link Link4: mass 0.289633681619295 -> 0.685
- link Link5: mass 0.239419768320061 -> 0.619
- link Link6: mass 0.218799761431682 -> 0.602
- link Link7: mass 0.0649018034311231 -> 0.107
- link base_link: mass 0.841071174772543 -> 1.862

File: rm_description/urdf/rm_75_6f.urdf (robot description, URDF)
Before this commit: robot rm_75_6f_description, 8 links, 7 joints
Links:
- link Link1: mass 0.59356 -> 1.574
- link Link2: mass 0.43285 -> 1.217
- link Link3: mass 0.43132 -> 1.11
- link Link4: mass 0.28963 -> 0.685
- link Link5: mass 0.23941 -> 0.619
- link Link6: mass 0.21879 -> 0.602
- link Link7: mass 0.14433 -> 0.144
- link base_link: mass 0.84105 -> 1.862

File: rm_description/urdf/rm_75_6fb.urdf (robot description, URDF)
Before this commit: robot RM75-6F, 8 links, 7 joints
Links:
- link Link7: mass 3.04449097310784 -> 0.144
- link Link_1: mass 0.593542243994357 -> 1.574
- link Link_2: mass 0.432849544766671 -> 1.217
- link Link_3: mass 0.431326296657269 -> 1.11
- link Link_4: mass 0.289643824188822 -> 0.685
- link Link_5: mass 0.239430992940448 -> 0.619
- link Link_6: mass 0.21879527056675 -> 0.602
- link base_link: mass 0.838885280844642 -> 1.862

File: rm_description/urdf/rm_eco62.urdf (robot description, URDF)
Before this commit: robot rm_eco62, 7 links, 6 joints
Links:
- link link_1: mass 0.384569120432882 -> 1.19575
- link link_2: mass 1.33623855048231 -> 0.8055
- link link_3: mass 0.332154099628179 -> 0.413
- link link_4: mass 0.110752178156894 -> 0.2386
- link link_5: mass 0.153716854003785 -> 0.2633
- link link_6: mass 0.0471960682349858 -> 0.0667

File: rm_description/urdf/rm_eco63.urdf (robot description, URDF)
Before this commit: robot rm_eco63, 8 links, 7 joints
Links:
- link Link1: mass 0.656374618338142 -> 1.6026
- link Link2: mass 5.26262523683375 -> 2.8169
- link Link3: mass 1.3509329667983 -> 2.6857
- link Link4: mass 0.733001235394853 -> 0.625
- link Link5: mass 0.911747774463918 -> 0.6743
- link Link6: mass 0.065035417997418 -> 0.248
- link base_link: mass 8.97974481667473 -> 1

File: rm_description/urdf/rm_eco63_6fb.urdf (robot description, URDF)
Before this commit: robot ECO63-6FB-URDF, 7 links, 6 joints
Links:
- link Link1: mass 0.656374618338142 -> 1.6026
- link Link2: mass 5.26262523683375 -> 2.8169
- link Link3: mass 1.3509329667983 -> 2.6857
- link Link4: mass 0.733001235394853 -> 0.625
- link Link5: mass 0.911747774463918 -> 0.6743
- link Link6: mass 0.151764173288042 -> 0.248
- link base_link: mass 9.06647326360739 -> 1

File: rm_description/urdf/rm_eco65_6f.urdf (robot description, URDF)
Before this commit: robot eco65, 7 links, 6 joints
Links:
- link Link1: mass 0.74252212802658 -> 1.507
- link Link2: mass 1.35020712394805 -> 2.0227
- link Link3: mass 1.0422213139163 -> 1.8858
- link Link4: mass 0.273792481713346 -> 0.57
- link Link5: mass 0.27793758472494 -> 0.641
- link Link6: mass 0.14611108984048 -> 0.0857

File: rm_description/urdf/rm_eco65_6fb.urdf (robot description, URDF)
Before this commit: robot 0000-eco65_URDF(2), 7 links, 6 joints
Links:
- link base_link: mass 1.6314377241954 -> 2
- link link1: mass 1.76684172446222 -> 1.507
- link link2: mass 3.5404490739212 -> 2.0227
- link link3: mass 2.66024465891583 -> 1.8858
- link link4: mass 0.733002748293818 -> 0.57
- link link5: mass 0.911746755408486 -> 0.641
- link link6: mass 0.305602477849543 -> 0.0857

File: rm_description/urdf/rm_rx75l-6fb.urdf (robot description, URDF)
Before this commit: robot RXL-6FB, 9 links, 8 joints
Links:
- link Link1: mass 0.851539025255045 -> 1.559
- link Link2: mass 0.870077465148622 -> 1.394
- link Link3: mass 0.593225766113055 -> 1.117
- link Link4: mass 0.395483565870343 -> 0.673
- link Link5: mass 0.845200261498234 -> 1.13
- link Link6: mass 0.280942850777542 -> 0.559
- link Link7: mass 0.23898 -> 0.483
- link Link8: mass 0.16582 -> 0.0
- link base_link: mass 0.651913537431184 -> 0.651913537431336

File: rm_description/urdf/rm_rx75r-6fb.urdf (robot description, URDF)
Before this commit: robot RXR-6FB, 9 links, 8 joints
Links:
- link Link1: mass 0.851539173063523 -> 1.559
- link Link2: mass 0.87008 -> 1.384
- link Link3: mass 0.593225765910811 -> 1.117
- link Link4: mass 0.395483546701072 -> 0.665
- link Link5: mass 0.845201652493134 -> 1.13
- link Link6: mass 0.280941853294711 -> 0.559
- link Link7: mass 0.229769882476631 -> 0.483
- link Link8: mass 0.165822947667674 -> 0.0
- link base_link: mass 0.651913537431336 -> 0.651913537431184

File: rm_description/urdf/rml_63.urdf (robot description, URDF)
Before this commit: robot rml_63_description, 7 links, 6 joints
Links:
- link base_link: mass 0.66248 -> 1.862
- link link1: mass 1.7668 -> 1.837
- link link2: mass 4.3415 -> 2.006
- link link3: mass 1.7286 -> 1.961
- link link4: mass 2.4734 -> 1.201
- link link5: mass 0.93162 -> 1.026
- link link6: mass 0.065037 -> 0.107

File: rm_description/urdf/rml_63_6f.urdf (robot description, URDF)
Before this commit: robot rm_63_6f_description, 7 links, 6 joints
Links:
- link Link1: mass 0.92308 -> 1.837
- link Link2: mass 1.5577 -> 2.006
- link Link3: mass 0.71556 -> 1.961
- link Link4: mass 0.69692 -> 1.201
- link Link5: mass 0.3567 -> 1.026
- link Link6: mass 0.14814 -> 0.248
- link base_link: mass 0.66248 -> 1.862

File: rm_description/urdf/rml_63_6fb.urdf (robot description, URDF)
Before this commit: robot RML-63-6F, 7 links, 6 joints
Links:
- link Link_1: mass 1.7668 -> 1.837
- link Link_2: mass 4.3415 -> 2.006
- link Link_3: mass 1.7286 -> 1.961
- link Link_4: mass 2.4734 -> 1.201
- link Link_5: mass 0.93162 -> 1.026
- link Link_6: mass 0.3056 -> 0.248
- link base_link: mass 1.6314 -> 1.862

Commit message: Sync URDF mass/inertia parameters from rm_models

File: rm_description/urdf/rm_65.urdf (robot description, URDF)
Before this commit: robot rm_65_description, 7 links, 6 joints
Links:
- link Link1: mass 0.593563443690403 -> 1.51
- link Link2: mass 0.864175046869043 -> 1.653
- link Link3: mass 0.289633681624654 -> 0.726
- link Link4: mass 0.239419768320061 -> 0.671
- link Link5: mass 0.218799761431678 -> 0.647
- link Link6: mass 0.0649018034311231 -> 0.104
- link base_link: mass 0.841070778135659 -> 1.862

File: rm_description/urdf/rm_eco63.urdf (robot description, URDF)
Before this commit: robot rm_eco63, 8 links, 7 joints
Links:
- link Link1: mass 0.656374618338142 -> 1.6026
- link Link2: mass 5.26262523683375 -> 2.8169
- link Link3: mass 1.3509329667983 -> 2.6857
- link Link4: mass 0.733001235394853 -> 0.625
- link Link5: mass 0.911747774463918 -> 0.6743
- link Link6: mass 0.065035417997418 -> 0.248
- link base_link: mass 8.97974481667473 -> 1

Commit message: Update URDF files from humble directory

File: rm_description/urdf/rm_65.urdf (robot description, URDF)
Before this commit: robot rm_65_description, 7 links, 6 joints
Links:
- link Link1: mass 1.51 -> 0.593563443690403
- link Link2: mass 1.653 -> 0.864175046869043
- link Link3: mass 0.726 -> 0.289633681624654
- link Link4: mass 0.671 -> 0.239419768320061
- link Link5: mass 0.647 -> 0.218799761431678
- link Link6: mass 0.104 -> 0.0649018034311231
- link base_link: mass 1.862 -> 0.841070778135659

File: rm_description/urdf/rm_65_6f.urdf (robot description, URDF)
Before this commit: robot rm_65_6f_description, 7 links, 6 joints
Links:
- link Link1: mass 1.51 -> 0.59356
- link Link2: mass 1.653 -> 0.86418
- link Link3: mass 0.726 -> 0.28963
- link Link4: mass 0.671 -> 0.23941
- link Link5: mass 0.647 -> 0.21879
- link Link6: mass 0.14434 -> 0.14433
- link base_link: mass 1.862 -> 0.84105

File: rm_description/urdf/rm_65_6fb.urdf (robot description, URDF)
Before this commit: robot RM65-6F, 7 links, 6 joints
Links:
- link Link1: mass 1.51 -> 0.593542243994357
- link Link2: mass 1.653 -> 0.86417584142394
- link Link3: mass 0.726 -> 0.289643824525119
- link Link4: mass 0.671 -> 0.239430992940448
- link Link5: mass 0.647 -> 0.21879527056675
- link Link6: mass 0.14434 -> 3.04449097371379
- link base_link: mass 1.862 -> 0.838885281114303

File: rm_description/urdf/rm_75.urdf (robot description, URDF)
Before this commit: robot rm_75_description, 8 links, 7 joints
Links:
- link Link1: mass 1.574 -> 0.593563458735581
- link Link2: mass 1.217 -> 0.432849770310974
- link Link3: mass 1.11 -> 0.431325495678459
- link Link4: mass 0.685 -> 0.289633681619295
- link Link5: mass 0.619 -> 0.239419768320061
- link Link6: mass 0.602 -> 0.218799761431682
- link Link7: mass 0.107 -> 0.0649018034311231
- link base_link: mass 1.862 -> 0.841071174772543

File: rm_description/urdf/rm_75_6f.urdf (robot description, URDF)
Before this commit: robot rm_75_6f_description, 8 links, 7 joints
Links:
- link Link1: mass 1.574 -> 0.59356
- link Link2: mass 1.217 -> 0.43285
- link Link3: mass 1.11 -> 0.43132
- link Link4: mass 0.685 -> 0.28963
- link Link5: mass 0.619 -> 0.23941
- link Link6: mass 0.602 -> 0.21879
- link Link7: mass 0.144 -> 0.14433
- link base_link: mass 1.862 -> 0.84105

File: rm_description/urdf/rm_75_6fb.urdf (robot description, URDF)
Before this commit: robot RM75-6F, 8 links, 7 joints
Links:
- link Link7: mass 0.144 -> 3.04449097310784
- link Link_1: mass 1.574 -> 0.593542243994357
- link Link_2: mass 1.217 -> 0.432849544766671
- link Link_3: mass 1.11 -> 0.431326296657269
- link Link_4: mass 0.685 -> 0.289643824188822
- link Link_5: mass 0.619 -> 0.239430992940448
- link Link_6: mass 0.602 -> 0.21879527056675
- link base_link: mass 1.862 -> 0.838885280844642

File: rm_description/urdf/rm_eco62.urdf (robot description, URDF)
Before this commit: robot rm_eco62, 7 links, 6 joints
Links:
- link link_1: mass 1.19575 -> 0.384569120432882
- link link_2: mass 0.8055 -> 1.33623855048231
- link link_3: mass 0.413 -> 0.332154099628179
- link link_4: mass 0.2386 -> 0.110752178156894
- link link_5: mass 0.2633 -> 0.153716854003785
- link link_6: mass 0.0667 -> 0.0471960682349858

File: rm_description/urdf/rm_eco63.urdf (robot description, URDF)
Before this commit: robot rm_eco63, 8 links, 7 joints
Links:
- link Link1: mass 1.6026 -> 0.656374618338142
- link Link2: mass 2.8169 -> 5.26262523683375
- link Link3: mass 2.6857 -> 1.3509329667983
- link Link4: mass 0.625 -> 0.733001235394853
- link Link5: mass 0.6743 -> 0.911747774463918
- link Link6: mass 0.248 -> 0.065035417997418
- link base_link: mass 1 -> 8.97974481667473

File: rm_description/urdf/rm_eco63_6fb.urdf (robot description, URDF)
Before this commit: robot ECO63-6FB-URDF, 7 links, 6 joints
Links:
- link Link1: mass 1.6026 -> 0.656374618338142
- link Link2: mass 2.8169 -> 5.26262523683375
- link Link3: mass 2.6857 -> 1.3509329667983
- link Link4: mass 0.625 -> 0.733001235394853
- link Link5: mass 0.6743 -> 0.911747774463918
- link Link6: mass 0.248 -> 0.151764173288042
- link base_link: mass 1 -> 9.06647326360739

File: rm_description/urdf/rm_eco65_6f.urdf (robot description, URDF)
Before this commit: robot eco65, 7 links, 6 joints
Links:
- link Link1: mass 1.507 -> 0.74252212802658
- link Link2: mass 2.0227 -> 1.35020712394805
- link Link3: mass 1.8858 -> 1.0422213139163
- link Link4: mass 0.57 -> 0.273792481713346
- link Link5: mass 0.641 -> 0.27793758472494
- link Link6: mass 0.0857 -> 0.14611108984048

File: rm_description/urdf/rm_eco65_6fb.urdf (robot description, URDF)
Before this commit: robot 0000-eco65_URDF(2), 7 links, 6 joints
Links:
- link base_link: mass 2 -> 1.6314377241954
- link link1: mass 1.507 -> 1.76684172446222
- link link2: mass 2.0227 -> 3.5404490739212
- link link3: mass 1.8858 -> 2.66024465891583
- link link4: mass 0.57 -> 0.733002748293818
- link link5: mass 0.641 -> 0.911746755408486
- link link6: mass 0.0857 -> 0.305602477849543

File: rm_description/urdf/rm_rx75l-6fb.urdf (robot description, URDF)
Before this commit: robot RXL-6FB, 9 links, 8 joints
Links:
- link Link1: mass 1.559 -> 0.851539025255045
- link Link2: mass 1.394 -> 0.870077465148622
- link Link3: mass 1.117 -> 0.593225766113055
- link Link4: mass 0.673 -> 0.395483565870343
- link Link5: mass 1.13 -> 0.845200261498234
- link Link6: mass 0.559 -> 0.280942850777542
- link Link7: mass 0.483 -> 0.23898
- link Link8: mass 0.0 -> 0.16582
- link base_link: mass 0.651913537431336 -> 0.651913537431184

File: rm_description/urdf/rm_rx75r-6fb.urdf (robot description, URDF)
Before this commit: robot RXR-6FB, 9 links, 8 joints
Links:
- link Link1: mass 1.559 -> 0.851539173063523
- link Link2: mass 1.384 -> 0.87008
- link Link3: mass 1.117 -> 0.593225765910811
- link Link4: mass 0.665 -> 0.395483546701072
- link Link5: mass 1.13 -> 0.845201652493134
- link Link6: mass 0.559 -> 0.280941853294711
- link Link7: mass 0.483 -> 0.229769882476631
- link Link8: mass 0.0 -> 0.165822947667674
- link base_link: mass 0.651913537431184 -> 0.651913537431336

File: rm_description/urdf/rml_63.urdf (robot description, URDF)
Before this commit: robot rml_63_description, 7 links, 6 joints
Links:
- link base_link: mass 1.862 -> 0.66248
- link link1: mass 1.837 -> 1.7668
- link link2: mass 2.006 -> 4.3415
- link link3: mass 1.961 -> 1.7286
- link link4: mass 1.201 -> 2.4734
- link link5: mass 1.026 -> 0.93162
- link link6: mass 0.107 -> 0.065037

File: rm_description/urdf/rml_63_6f.urdf (robot description, URDF)
Before this commit: robot rm_63_6f_description, 7 links, 6 joints
Links:
- link Link1: mass 1.837 -> 0.92308
- link Link2: mass 2.006 -> 1.5577
- link Link3: mass 1.961 -> 0.71556
- link Link4: mass 1.201 -> 0.69692
- link Link5: mass 1.026 -> 0.3567
- link Link6: mass 0.248 -> 0.14814
- link base_link: mass 1.862 -> 0.66248

File: rm_description/urdf/rml_63_6fb.urdf (robot description, URDF)
Before this commit: robot RML-63-6F, 7 links, 6 joints
Links:
- link Link_1: mass 1.837 -> 1.7668
- link Link_2: mass 2.006 -> 4.3415
- link Link_3: mass 1.961 -> 1.7286
- link Link_4: mass 1.201 -> 2.4734
- link Link_5: mass 1.026 -> 0.93162
- link Link_6: mass 0.248 -> 0.3056
- link base_link: mass 1.862 -> 1.6314

Commit message: Update code from jazzy directory

File: rm_description/urdf/rm_65.urdf (robot description, URDF)
Before this commit: robot rm_65_description, 7 links, 6 joints
Links:
- link Link1: mass 1.51 -> 0.593563443690403
- link Link2: mass 1.653 -> 0.864175046869043
- link Link3: mass 0.726 -> 0.289633681624654
- link Link4: mass 0.671 -> 0.239419768320061
- link Link5: mass 0.647 -> 0.218799761431678
- link Link6: mass 0.104 -> 0.0649018034311231
- link base_link: mass 1.862 -> 0.841070778135659
