Commit message: fix: 修正模型惯量数据

File: rm_description/urdf/imported/eco65_6f.urdf.xacro (robot description, xacro)
@@ -100,7 +100,7 @@
   <link name="Link4">
     <inertial>
-      <origin rpy="0 0 0" xyz="-0.0069819 -0.016328 0.0067416" />
-      <mass value="0.27383" />
-      <inertia ixx="0.00024751" ixy="-5.6849E-09" ixz="5.4838E-10" iyy="0.00017648" iyz="-2.8552E-05" izz="0.00019295" />
+      <origin rpy="0 0 0" xyz="1.1437E-07 -0.0098794 0.013445" />
+      <mass value="0.27261" />
+      <inertia ixx="0.00023835" ixy="1.6845E-09" ixz="6.2757E-09" iyy="0.00019072" iyz="4.0013E-05" izz="0.0001713" />
     </inertial>
     <collision>

File: rm_description/urdf/imported/eco65_6fb.urdf.xacro (robot description, xacro)
@@ -100,7 +100,7 @@
   <link name="Link4">
     <inertial>
-      <origin rpy="0 0 0" xyz="-0.0069819 -0.016328 0.0067416" />
-      <mass value="0.27383" />
-      <inertia ixx="0.00024751" ixy="-5.6849E-09" ixz="5.4838E-10" iyy="0.00017648" iyz="-2.8552E-05" izz="0.00019295" />
+      <origin rpy="0 0 0" xyz="1.1437E-07 -0.0098794 0.013445" />
+      <mass value="0.27261" />
+      <inertia ixx="0.00023835" ixy="1.6845E-09" ixz="6.2757E-09" iyy="0.00019072" iyz="4.0013E-05" izz="0.0001713" />
     </inertial>
     <collision>

File: rm_description/urdf/imported/eco65_standard.urdf.xacro (robot description, xacro)
@@ -100,7 +100,7 @@
   <link name="Link4">
     <inertial>
-      <origin rpy="0 0 0" xyz="-4.028E-05 -3.496E-02 3.8015E-03" />
-      <mass value="0.57" />
-      <inertia ixx="4.97615E-04" ixy="5.3887E-07" ixz="7.046E-07" iyy="3.2497E-04" iyz="0" izz="1.1634E-03" />
+      <origin rpy="0 0 0" xyz="1.1437E-07 -0.0098794 0.013445" />
+      <mass value="0.27261" />
+      <inertia ixx="0.00023835" ixy="1.6845E-09" ixz="6.2757E-09" iyy="0.00019072" iyz="4.0013E-05" izz="0.0001713" />
     </inertial>
     <collision>

File: rm_description/urdf/rm_eco62_gazebo.urdf (robot description, URDF)
Before this commit: robot rm_eco62_description, 7 links, 6 joints
Links:
- link Link1: mass 1.19575 -> 0.384569120432882
- link Link4: mass 0.2386 -> 0.110752178156894

File: rm_description/urdf/rm_eco62_gazebo.urdf.xacro (robot description, xacro)
@@ -27,7 +27,7 @@
   <link name="Link1">
     <inertial>
-      <origin xyz="-0.036 -0.01347 -0.00908" rpy="0 0 0" />
-      <mass value="1.19575" />
-      <inertia ixx="0.01026" ixy="0.000561" ixz="-0.000395" iyy="0.002074" iyz="-0.00145" izz="0.02213" />
+      <origin xyz="-0.0382156936663754 -0.00545476263009575 -0.00248189073126664" rpy="0 0 0" />
+      <mass value="0.384569120432882" />
+      <inertia ixx="0.00022257753835175" ixy="-7.70372317374323E-05" ixz="4.37635506114307E-05" iyy="0.000605579716850644" iyz="4.05126631912246E-06" izz="0.000631817968488901" />
     </inertial>
     <visual>
@@ -114,7 +114,7 @@
   <link name="Link4">
     <inertial>
-      <origin xyz="0 -0.0168 0.0034" rpy="0 0 0" />
-      <mass value="0.2386" />
-      <inertia ixx="0.000965" ixy="0" ixz="0" iyy="0.0000704" iyz="0.0000144" izz="0.0000915" />
+      <origin xyz="1.37711279149522E-06 -0.009725196668249 0.00396013823109714" rpy="0 0 0" />
+      <mass value="0.110752178156894" />
+      <inertia ixx="4.91297766773849E-05" ixy="1.12199756370538E-09" ixz="-1.03735450320981E-09" iyy="3.42721993306208E-05" iyz="-5.21925020486496E-06" izz="4.57514364497173E-05" />
     </inertial>
     <visual>

File: rm_description/urdf/rm_eco65.urdf (robot description, URDF)
Before this commit: robot rm_eco65_description, 7 links, 6 joints
Links:
- link Link4: mass 0.57 -> 0.27261

File: rm_description/urdf/rm_eco65.urdf.xacro (robot description, xacro)
@@ -223,15 +223,15 @@
     <inertial>
       <origin
-        xyz="-0.0069819 -0.016328 0.0067416"
+        xyz="1.1437E-07 -0.0098794 0.013445"
         rpy="0 0 0" />
       <mass
-        value="0.27383" />
+        value="0.27261" />
       <inertia
-        ixx="0.00024751"
-        ixy="-5.6849E-09"
-        ixz="5.4838E-10"
-        iyy="0.00017648"
-        iyz="-2.8552E-05"
-        izz="0.00019295"/>
+        ixx="0.00023835"
+        ixy="1.6845E-09"
+        ixz="6.2757E-09"
+        iyy="0.00019072"
+        iyz="4.0013E-05"
+        izz="0.0001713"/>
     </inertial>
     <visual>

File: rm_description/urdf/rm_eco65_6f.urdf (robot description, URDF)
Before this commit: robot eco65, 7 links, 6 joints
Links:
- link Link4: mass 0.57 -> 0.27261

File: rm_description/urdf/rm_eco65_6fb.urdf (robot description, URDF)
Before this commit: robot 0000-eco65_URDF(2), 7 links, 6 joints
Links:
- link link4: mass 0.57 -> 0.27261

File: rm_description/urdf/rm_eco65_gazebo.urdf (robot description, URDF)
Before this commit: robot rm_eco65_description, 7 links, 6 joints
Links:
- link Link4: mass 0.57 -> 0.27261

File: rm_description/urdf/rm_eco65_gazebo.urdf.xacro (robot description, xacro)
@@ -223,15 +223,15 @@
     <inertial>
       <origin
-        xyz="-0.0069819 -0.016328 0.0067416"
+        xyz="1.1437E-07 -0.0098794 0.013445"
         rpy="0 0 0" />
       <mass
-        value="0.27383" />
+        value="0.27261" />
       <inertia
-        ixx="0.00024751"
-        ixy="-5.6849E-09"
-        ixz="5.4838E-10"
-        iyy="0.00017648"
-        iyz="-2.8552E-05"
-        izz="0.00019295"/>
+        ixx="0.00023835"
+        ixy="1.6845E-09"
+        ixz="6.2757E-09"
+        iyy="0.00019072"
+        iyz="4.0013E-05"
+        izz="0.0001713"/>
     </inertial>
     <visual>

Commit message: fix: 修正模型惯量数据

File: rm_description/urdf/imported/eco65_6f.urdf.xacro (robot description, xacro)
@@ -100,7 +100,7 @@
   <link name="Link4">
     <inertial>
-      <origin rpy="0 0 0" xyz="-0.0069819 -0.016328 0.0067416" />
-      <mass value="0.27383" />
-      <inertia ixx="0.00024751" ixy="-5.6849E-09" ixz="5.4838E-10" iyy="0.00017648" iyz="-2.8552E-05" izz="0.00019295" />
+      <origin rpy="0 0 0" xyz="1.1437E-07 -0.0098794 0.013445" />
+      <mass value="0.27261" />
+      <inertia ixx="0.00023835" ixy="1.6845E-09" ixz="6.2757E-09" iyy="0.00019072" iyz="4.0013E-05" izz="0.0001713" />
     </inertial>
     <collision>

File: rm_description/urdf/imported/eco65_6fb.urdf.xacro (robot description, xacro)
@@ -100,7 +100,7 @@
   <link name="Link4">
     <inertial>
-      <origin rpy="0 0 0" xyz="-0.0069819 -0.016328 0.0067416" />
-      <mass value="0.27383" />
-      <inertia ixx="0.00024751" ixy="-5.6849E-09" ixz="5.4838E-10" iyy="0.00017648" iyz="-2.8552E-05" izz="0.00019295" />
+      <origin rpy="0 0 0" xyz="1.1437E-07 -0.0098794 0.013445" />
+      <mass value="0.27261" />
+      <inertia ixx="0.00023835" ixy="1.6845E-09" ixz="6.2757E-09" iyy="0.00019072" iyz="4.0013E-05" izz="0.0001713" />
     </inertial>
     <collision>

File: rm_description/urdf/imported/eco65_standard.urdf.xacro (robot description, xacro)
@@ -100,7 +100,7 @@
   <link name="Link4">
     <inertial>
-      <origin rpy="0 0 0" xyz="-4.028E-05 -3.496E-02 3.8015E-03" />
-      <mass value="0.57" />
-      <inertia ixx="4.97615E-04" ixy="5.3887E-07" ixz="7.046E-07" iyy="3.2497E-04" iyz="0" izz="1.1634E-03" />
+      <origin rpy="0 0 0" xyz="1.1437E-07 -0.0098794 0.013445" />
+      <mass value="0.27261" />
+      <inertia ixx="0.00023835" ixy="1.6845E-09" ixz="6.2757E-09" iyy="0.00019072" iyz="4.0013E-05" izz="0.0001713" />
     </inertial>
     <collision>

File: rm_description/urdf/rm_75_gazebo.urdf.xacro (robot description, xacro)
@@ -14,10 +14,10 @@
         value="0.841071174772543" />
       <inertia
-        ixx="0"
-        ixy="0"
-        ixz="0"
-        iyy="0"
-        iyz="0"
-        izz="0" />
+        ixx="0.00172611149818605"
+        ixy="2.52724703312125E-06"
+        ixz="3.67689528877993E-05"
+        iyy="0.00170987425756066"
+        iyz="-1.68009023667311E-06"
+        izz="0.000904023916742301" />
     </inertial>
     <visual>
@@ -54,10 +54,10 @@
         value="0.593563458735581" />
       <inertia
-        ixx="0"
-        ixy="0"
-        ixz="0"
-        iyy="0"
-        iyz="0"
-        izz="0" />
+        ixx="0.000561352422092522"
+        ixy="9.8019294192418E-09"
+        ixz="-0.000211217278563478"
+        iyy="0.00126614121202124"
+        iyz="1.29510293158304E-08"
+        izz="0.0011816817861243" />
     </inertial>
     <visual>
@@ -112,10 +112,10 @@
         value="0.432849770310974" />
       <inertia
-        ixx="0"
-        ixy="0"
-        ixz="0"
-        iyy="0"
-        iyz="0"
-        izz="0" />
+        ixx="0.00125838173873093"
+        ixy="5.63146579602116E-09"
+        ixz="1.33486683063366E-09"
+        iyy="0.00122245448121472"
+        iyz="0.000279003475762058"
+        izz="0.000317474184276672" />
     </inertial>
     <visual>
@@ -170,10 +170,10 @@
         value="0.431325495678459" />
       <inertia
-        ixx="0"
-        ixy="0"
-        ixz="0"
-        iyy="0"
-        iyz="0"
-        izz="0" />
+        ixx="0.000794332771462568"
+        ixy="1.03353218375171E-08"
+        ixz="-2.32798826854953E-09"
+        iyy="0.000315065343266245"
+        iyz="-0.000142620540462618"
+        izz="0.000730371131605455" />
     </inertial>
     <visual>
@@ -228,10 +228,10 @@
         value="0.289633681619295" />
       <inertia
-        ixx="0"
-        ixy="0"
-        ixz="0"
-        iyy="0"
-        iyz="0"
-        izz="0" />
+        ixx="0.000637371004484591"
+        ixy="-3.86643270900744E-08"
+        ixz="7.05261290886955E-08"
+        iyy="0.000614178164759844"
+        iyz="0.000144610359942128"
+        izz="0.000156483880946498" />
     </inertial>
     <visual>
@@ -286,10 +286,10 @@
         value="0.239419768320061" />
       <inertia
-        ixx="0"
-        ixy="0"
-        ixz="0"
-        iyy="0"
-        iyz="0"
-        izz="0" />
+        ixx="0.000285938919722783"
+        ixy="2.21994116852616E-09"
+        ixz="3.07101358617598E-09"
+        iyy="0.00011988808279186"
+        iyz="-4.4236583260078E-05"
+        izz="0.000262727540304212" />
     </inertial>
     <visual>
@@ -344,10 +344,10 @@
         value="0.218799761431682" />
       <inertia
-        ixx="0"
-        ixy="0"
-        ixz="0"
-        iyy="0"
-        iyz="0"
-        izz="0" />
+        ixx="0.000350540363914436"
+        ixy="-1.7705645712277E-08"
+        ixz="3.41781620449632E-08"
+        iyy="0.000334482418423991"
+        iyz="7.82431228462317E-05"
+        izz="0.000104927867487584" />
     </inertial>
     <visual>
@@ -403,10 +403,10 @@
         value="0.0649018034311231" />
       <inertia
-        ixx="0"
-        ixy="0"
-        ixz="0"
-        iyy="0"
-        iyz="0"
-        izz="0" />
+        ixx="2.02766547502765E-05"
+        ixy="-1.32505200276848E-06"
+        ixz="-2.58450915224912E-08"
+        iyy="1.87986725225022E-05"
+        iyz="3.39471452123283E-09"
+        izz="3.17885459163081E-05" />
     </inertial>
     <visual>
@@ -463,10 +463,10 @@
         value="0.14433" />
       <inertia
-        ixx="0"
-        ixy="0"
-        ixz="0"
-        iyy="0"
-        iyz="0"
-        izz="0" />
+        ixx="3.6119E-05"
+        ixy="-1.3242E-06"
+        ixz="-3.2733E-08"
+        iyy="3.4626E-05"
+        iyz="7.6694E-09"
+        izz="6.1463E-05" />
     </inertial>
     <visual>
@@ -523,10 +523,10 @@
         value="3.04449097310784" />
       <inertia
-        ixx="0"
-        ixy="0"
-        ixz="0"
-        iyy="0"
-        iyz="0"
-        izz="0" />
+        ixx="0.17081032825412"
+        ixy="5.38227954656055E-07"
+        ixz="0.000151207463266663"
+        iyy="0.169967421488281"
+        iyz="0.0010577717307003"
+        izz="0.0030554606628762" />
     </inertial>
     <visual>

File: rm_description/urdf/rm_eco62_gazebo.urdf.xacro (robot description, xacro)
@@ -7,5 +7,5 @@
       <origin xyz="0.00133682761157797 -8.82763422017089E-05 0.0439834418774717" rpy="0 0 0" />
       <mass value="0.584825481285431" />
-      <inertia ixx="0" ixy="0" ixz="0" iyy="0" iyz="0" izz="0" />
+      <inertia ixx="0.000775925119945014" ixy="2.98148797430621E-06" ixz="-2.52746653512818E-05" iyy="0.000790075378837822" iyz="2.12739218651747E-06" izz="0.000587764326506914" />
     </inertial>
     <visual>
@@ -29,5 +29,5 @@
       <origin xyz="-0.0382156936663754 -0.00545476263009575 -0.00248189073126664" rpy="0 0 0" />
       <mass value="0.384569120432882" />
-      <inertia ixx="0" ixy="0" ixz="0" iyy="0" iyz="0" izz="0" />
+      <inertia ixx="0.00022257753835175" ixy="-7.70372317374323E-05" ixz="4.37635506114307E-05" iyy="0.000605579716850644" iyz="4.05126631912246E-06" izz="0.000631817968488901" />
     </inertial>
     <visual>
@@ -58,5 +58,5 @@
       <origin xyz="0.0876574260013383 7.06115941204177E-07 -0.0582757120216016" rpy="0 0 0" />
       <mass value="1.33623855048231" />
-      <inertia ixx="0" ixy="0" ixz="0" iyy="0" iyz="0" izz="0" />
+      <inertia ixx="0.000782439324383488" ixy="3.30138611119598E-08" ixz="-0.000592670610886331" iyy="0.00567774731360305" iyz="-1.48333937024788E-08" izz="0.0056479745580982" />
     </inertial>
     <visual>
@@ -87,5 +87,5 @@
       <origin xyz="0.064390668361978 1.69820375292562E-06 0.00482231553499824" rpy="0 0 0" />
       <mass value="0.332154099628179" />
-      <inertia ixx="0" ixy="0" ixz="0" iyy="0" iyz="0" izz="0" />
+      <inertia ixx="0.000128065855853166" ixy="3.73125577149301E-09" ixz="5.57695241071185E-05" iyy="0.00114220860014717" iyz="-1.28387853936544E-09" izz="0.00116351274597718" />
     </inertial>
     <visual>
@@ -116,5 +116,5 @@
       <origin xyz="1.37711279149522E-06 -0.009725196668249 0.00396013823109714" rpy="0 0 0" />
       <mass value="0.110752178156894" />
-      <inertia ixx="0" ixy="0" ixz="0" iyy="0" iyz="0" izz="0" />
+      <inertia ixx="4.91297766773849E-05" ixy="1.12199756370538E-09" ixz="-1.03735450320981E-09" iyy="3.42721993306208E-05" iyz="-5.21925020486496E-06" izz="4.57514364497173E-05" />
     </inertial>
     <visual>
@@ -145,5 +145,5 @@
       <origin xyz="5.08842681060107E-07 0.00420077719178583 -0.00358941394658707" rpy="0 0 0" />
       <mass value="0.153716854003785" />
-      <inertia ixx="0" ixy="0" ixz="0" iyy="0" iyz="0" izz="0" />
+      <inertia ixx="9.76286576153493E-05" ixy="-5.77416162886506E-09" ixz="1.60382177530514E-09" iyy="5.13289975047188E-05" iyz="-2.87378837336067E-06" izz="9.08724519634991E-05" />
     </inertial>
     <visual>
@@ -175,5 +175,5 @@
       <origin xyz="-7.72448794437025E-05 -2.38414868461989E-05 -0.0139344966930892" rpy="0 0 0" />
       <mass value="0.0471960682349858" />
-      <inertia ixx="0" ixy="0" ixz="0" iyy="0" iyz="0" izz="0" />
+      <inertia ixx="9.48227136591617E-06" ixy="5.23848349048734E-09" ixz="1.6103674761691E-08" iyy="9.4363237926155E-06" iyz="1.3729123698332E-08" izz="1.30412862089912E-05" />
     </inertial>
     <visual>

File: rm_description/urdf/rm_eco65.urdf (robot description, URDF)
Before this commit: robot rm_eco65_description, 7 links, 6 joints
Links:
- link Link4: mass 0.57 -> 0.27261

File: rm_description/urdf/rm_eco65.urdf.xacro (robot description, xacro)
@@ -223,15 +223,15 @@
     <inertial>
       <origin
-        xyz="-0.0069819 -0.016328 0.0067416"
+        xyz="1.1437E-07 -0.0098794 0.013445"
         rpy="0 0 0" />
       <mass
-        value="0.27383" />
+        value="0.27261" />
       <inertia
-        ixx="0.00024751"
-        ixy="-5.6849E-09"
-        ixz="5.4838E-10"
-        iyy="0.00017648"
-        iyz="-2.8552E-05"
-        izz="0.00019295"/>
+        ixx="0.00023835"
+        ixy="1.6845E-09"
+        ixz="6.2757E-09"
+        iyy="0.00019072"
+        iyz="4.0013E-05"
+        izz="0.0001713"/>
     </inertial>
     <visual>

File: rm_description/urdf/rm_eco65_6f.urdf (robot description, URDF)
Before this commit: robot eco65, 7 links, 6 joints
Links:
- link Link4: mass 0.57 -> 0.27261

File: rm_description/urdf/rm_eco65_6fb.urdf (robot description, URDF)
Before this commit: robot 0000-eco65_URDF(2), 7 links, 6 joints
Links:
- link link4: mass 0.57 -> 0.27261

File: rm_description/urdf/rm_eco65_gazebo.urdf (robot description, URDF)
Before this commit: robot rm_eco65_description, 7 links, 6 joints
Links:
- link Link4: mass 0.27383 -> 0.27261

File: rm_description/urdf/rm_eco65_gazebo.urdf.xacro (robot description, xacro)
@@ -223,15 +223,15 @@
     <inertial>
       <origin
-        xyz="-0.0069819 -0.016328 0.0067416"
+        xyz="1.1437E-07 -0.0098794 0.013445"
         rpy="0 0 0" />
       <mass
-        value="0.27383" />
+        value="0.27261" />
       <inertia
-        ixx="0.00024751"
-        ixy="-5.6849E-09"
-        ixz="5.4838E-10"
-        iyy="0.00017648"
-        iyz="-2.8552E-05"
-        izz="0.00019295"/>
+        ixx="0.00023835"
+        ixy="1.6845E-09"
+        ixz="6.2757E-09"
+        iyy="0.00019072"
+        iyz="4.0013E-05"
+        izz="0.0001713"/>
     </inertial>
     <visual>

File: rm_description/urdf/rml_63_gazebo.urdf.xacro (robot description, xacro)
@@ -216,10 +216,10 @@
         value="4.3415" />
       <inertia
-        ixx="0"
-        ixy="0"
-        ixz="0"
-        iyy="0"
-        iyz="0"
-        izz="0" />
+        ixx="0.0028306"
+        ixy="3.3846E-07"
+        ixz="4.0484E-06"
+        iyy="0.075435"
+        iyz="-3.3974E-08"
+        izz="0.075923" />
     </inertial>
     <visual>
@@ -274,10 +274,10 @@
         value="1.7286" />
       <inertia
-        ixx="0"
-        ixy="0"
-        ixz="0"
-        iyy="0"
-        iyz="0"
-        izz="0" />
+        ixx="0.0014154"
+        ixy="0.00068025"
+        ixz="-0.00043307"
+        iyy="0.0026049"
+        iyz="0.00017201"
+        izz="0.0028551" />
     </inertial>
     <visual>
@@ -332,10 +332,10 @@
         value="2.4734" />
       <inertia
-        ixx="0"
-        ixy="0"
-        ixz="0"
-        iyy="0"
-        iyz="0"
-        izz="0" />i
+        ixx="0.02602"
+        ixy="-1.1659E-07"
+        ixz="3.1323E-07"
+        iyy="0.024375"
+        iyz="0.0061661"
+        izz="0.002958" />i
     </inertial>
     <visual>
@@ -390,10 +390,10 @@
         value="0.93162" />
       <inertia
-        ixx="0"
-        ixy="0"
-        ixz="0"
-        iyy="0"
-        iyz="0"
-        izz="0" />
+        ixx="0.0012563"
+        ixy="-1.8115E-08"
+        ixz="-2.4669E-09"
+        iyy="0.0005379"
+        iyz="-0.00017339"
+        izz="0.0011134" />
     </inertial>
     <visual>
@@ -449,10 +449,10 @@
         value="0.065037" />
       <inertia
-        ixx="0"
-        ixy="0"
-        ixz="0"
-        iyy="0"
-        iyz="0"
-        izz="0" />
+        ixx="2.1144E-05"
+        ixy="-2.2803E-08"
+        ixz="2.5415E-08"
+        iyy="1.8109E-05"
+        iyz="1.0256E-08"
+        izz="3.19E-05" />
     </inertial>
     <visual>
@@ -509,10 +509,10 @@
         value="0.14814" />
       <inertia
-        ixx="0"
-        ixy="0"
-        ixz="0"
-        iyy="0"
-        iyz="0"
-        izz="0" />
+        ixx="7.2093E-05"
+        ixy="-1.2989E-06"
+        ixz="7.9524E-07"
+        iyy="7.063E-05"
+        iyz="-4.3017E-07"
+        izz="6.2819E-05" />
     </inertial>
     <visual>
@@ -569,10 +569,10 @@
         value="0.3056" />
       <inertia
-        ixx="0"
-        ixy="0"
-        ixz="0"
-        iyy="0"
-        iyz="0"
-        izz="0" />
+        ixx="0.00011383"
+        ixy="-3.6531E-08"
+        ixz="-1.1422E-07"
+        iyy="0.00011469"
+        iyz="4.3479E-08"
+        izz="0.00012619" />
     </inertial>
     <visual>
