Commit message: fix: 修复rm75-6f模型错误

File: rm_description/urdf/imported/75_6f.urdf.xacro (robot description, xacro)
@@ -196,5 +196,5 @@
   </link>
   <joint name="joint7" type="revolute">
-    <origin rpy="1.5708 0 0" xyz="0 -0.1725 0" />
+    <origin rpy="0 0 0" xyz="0 6.33627880320126e-07 0.172499999998836" />
     <parent link="Link6" />
     <child link="Link7" />

File: rm_description/urdf/rm_75.urdf.xacro (robot description, xacro)
@@ -498,6 +498,6 @@
     type="revolute">
     <origin
-      xyz="0 -0.1725 0"
-      rpy="1.5708 0 0" />
+      xyz="0 6.33627880320126e-07 0.172499999998836"
+      rpy="0 0 0" />
     <parent
       link="Link6" />

File: rm_description/urdf/rm_75_6f.urdf (robot description, URDF)
Before this commit: robot rm_75_6f_description, 8 links, 7 joints
Joints:
- joint joint7: origin xyz=0 -0.1725 0 rpy=1.5708 0 0 -> xyz=0 6.33627880320126e-07 0.172499999998836 rpy=0 0 0

File: rm_description/urdf/rm_75_gazebo.urdf.xacro (robot description, xacro)
@@ -498,6 +498,6 @@
     type="revolute">
     <origin
-      xyz="0 -0.1725 0"
-      rpy="1.5708 0 0" />
+      xyz="0 6.33627880320126e-07 0.172499999998836"
+      rpy="0 0 0" />
     <parent
       link="Link6" />
